Commit message: Changed ubi fingertip meshes and taxels, adapted distal phalanx to use them

File: sr_description/hand/xacro/finger/distal/distal.urdf.xacro (robot description, xacro)
@@ -1,9 +1,9 @@
 <robot xmlns:xacro="http://www.ros.org/wiki/xacro"
-xmlns:sensor="http://playerstage.sourceforge.net/gazebo/xmlschema/#sensor"
-xmlns:controller="http://playerstage.sourceforge.net/gazebo/xmlschema/#controller"
-xmlns:joint="http://playerstage.sourceforge.net/gazebo/xmlschema/#slider"
-xmlns:interface="http://playerstage.sourceforge.net/gazebo/xmlschema/#interface"
-xmlns:body="http://playerstage.sourceforge.net/gazebo/xmlschema/#body"
-xmlns:geom="http://playerstage.sourceforge.net/gazebo/xmlschema/#geom">
+       xmlns:sensor="http://playerstage.sourceforge.net/gazebo/xmlschema/#sensor"
+       xmlns:controller="http://playerstage.sourceforge.net/gazebo/xmlschema/#controller"
+       xmlns:joint="http://playerstage.sourceforge.net/gazebo/xmlschema/#slider"
+       xmlns:interface="http://playerstage.sourceforge.net/gazebo/xmlschema/#interface"
+       xmlns:body="http://playerstage.sourceforge.net/gazebo/xmlschema/#body"
+       xmlns:geom="http://playerstage.sourceforge.net/gazebo/xmlschema/#geom">
   <xacro:include filename="$(find sr_description)/hand/xacro/finger/distal/distal.gazebo.xacro" />
   <xacro:include filename="$(find sr_description)/hand/xacro/finger/distal/distal.transmission.xacro" />
@@ -30,5 +30,5 @@
         <geometry name="${prefix}${link_prefix}distal_visual">
           <xacro:if value="${ubi}">
-            <!-- Ubi distal -->
+			<!-- Ubi distal -->
             <mesh filename="package://sr_description/hand/model/ubi_tactiles/ubi_tip_visual.dae"
 		  scale="0.001 0.001 0.001" />
@@ -36,5 +36,5 @@
           <xacro:unless value="${ubi}">
             <xacro:if value="${eli}">
-              <!-- Ellispoid distal  -->
+							<!-- Ellispoid distal  -->
               <mesh filename="package://sr_description/hand/model/ellipsoids/distal_ellipsoid_visual.dae"
 		    scale="0.001 0.001 0.001" />
@@ -42,5 +42,5 @@
             <xacro:unless value="${eli}">
               <xacro:if value="${bio}">
-                <!-- biotac distal  -->
+				<!-- biotac distal  -->
                 <mesh filename="package://sr_description/hand/model/F1.dae"
                       scale="0.001 0.001 0.001" />
@@ -52,5 +52,5 @@
 		</xacro:if>
 		<xacro:unless value="${bt_sp}">
-                  <!-- Standard distal  -->
+				 <!-- Standard distal  -->
                   <mesh filename="package://sr_description/hand/model/F1.dae"
 			scale="0.001 0.001 0.001" />
@@ -66,5 +66,5 @@
         <geometry name="${prefix}${link_prefix}distal_collision_geom">
           <xacro:if value="${ubi}">
-            <!-- Ubi distal -->
+						<!-- Ubi distal -->
             <mesh filename="package://sr_description/hand/model/ubi_tactiles/ubi_tip_collision.dae"
             scale="0.001 0.001 0.001" />
@@ -72,5 +72,5 @@
           <xacro:unless value="${ubi}">
             <xacro:if value="${eli}">
-              <!-- Ellispoid distal  -->
+							<!-- Ellispoid distal  -->
               <mesh filename="package://sr_description/hand/model/ellipsoids/distal_ellipsoid.dae"
               scale="0.001 0.001 0.001" />
@@ -78,5 +78,5 @@
             <xacro:unless value="${eli}">
               <xacro:if value="${bio}">
-                <!-- biotac distal  -->
+								<!-- biotac distal  -->
                 <mesh filename="package://sr_description/hand/model/F1.dae"
                 scale="0.001 0.001 0.001" />
@@ -88,5 +88,5 @@
 		</xacro:if>
 		<xacro:unless value="${bt_sp}">
-                  <!-- Standard distal  -->
+								<!-- Standard distal  -->
                   <mesh filename="package://sr_description/hand/model/F1.dae"
 			scale="0.001 0.001 0.001" />
@@ -99,37 +99,37 @@
     </link>
     <xacro:unless value="${bio}">
-      <joint name="${prefix}${joint_prefix}J1" type="revolute">
+    <joint name="${prefix}${joint_prefix}J1" type="revolute">
         <parent link="${parent}" />
         <child link="${prefix}${link_prefix}distal" />
-        <origin xyz="0 0 0.025" rpy="0 0 0" />
-        <axis xyz="1 0 0" />
-        <xacro:if value="${bio}">
-          <!-- biotac fixed distal joint -->
+      <origin xyz="0 0 0.025" rpy="0 0 0" />
+      <axis xyz="1 0 0" />
+      <xacro:if value="${bio}">
+				<!-- biotac fixed distal joint -->
           <limit lower="${20/180*M_PI}" upper="${20/180*M_PI}"
           effort="10" velocity="2.0" />
         </xacro:if>
-        <xacro:unless value="${bio}">
-          <!-- standard distal joint -->
-          <limit lower="0" upper="${M_PI/2}" effort="2"
+      <xacro:unless value="${bio}">
+				<!-- standard distal joint -->
+        <limit lower="0" upper="${M_PI/2}" effort="2"
           velocity="2.0" />
         </xacro:unless>
         <dynamics damping="0.1" />
       </joint>
-      <gazebo reference="${prefix}${joint_prefix}J1">
-        <provideFeedback>1</provideFeedback>
-        <implicitSpringDamper>1</implicitSpringDamper>
+    <gazebo reference="${prefix}${joint_prefix}J1">
+      <provideFeedback>1</provideFeedback>
+      <implicitSpringDamper>1</implicitSpringDamper>
       </gazebo>
-      <link name="${prefix}${link_prefix}tip">
-        <inertial>
-          <mass value="0.001" />
+    <link name="${prefix}${link_prefix}tip">
+			<inertial>
+				<mass value="0.001" />
           <inertia ixx="0.0" ixy="0.0" ixz="0.0" iyy="0.0"
           iyz="0.0" izz="0.0" />
-        </inertial>
-      </link>
-      <joint name="${prefix}${joint_prefix}tip" type="fixed">
+  		</inertial>
+    </link>
+    <joint name="${prefix}${joint_prefix}tip" type="fixed">
         <parent link="${prefix}${link_prefix}distal" />
         <child link="${prefix}${link_prefix}tip" />
-        <origin xyz="0 0 0.026" rpy="0 0 0" />
-      </joint>
+      <origin xyz="0 0 0.026" rpy="0 0 0" />
+    </joint>
     </xacro:unless>
     <!-- extensions -->
