Commit message: Change sensor name in tactile plugin and tactile description Support namespace and use tactile plugin in distal sensors

File: sr_description/hand/xacro/finger/distal/distal.gazebo.xacro (robot description, xacro)
@@ -1,9 +1,9 @@
 <?xml version="1.0"?>
 <robot xmlns:xacro="http://www.ros.org/wiki/xacro">
-  <xacro:macro name="distal_gazebo" params="prefix link_prefix">
-  <!-- prefix can be anything but usually is "r_" or  "l_" for right and left hands distinction -->
+  <xacro:macro name="distal_gazebo" params="prefix link_prefix ns:=^|''">
+  <!-- prefix can be anything but usually is "rh_" or  "lh_" for right and left hands distinction -->
   <gazebo reference="${prefix}${link_prefix}distal">
-      <sensor type="contact" name="${prefix}${link_prefix}distal_contact">
-				<always_on>1</always_on>
+      <sensor type="contact" name="${prefix}${link_prefix}distal_sensor">
+        <always_on>1</always_on>
         <update_rate>1000.0</update_rate>
         <contact>
@@ -11,9 +11,11 @@
           <topic>${prefix}${link_prefix}distal_collision</topic>
         </contact>
-        <plugin name="${prefix}${link_prefix}distal_gazebo_ros_bumper_controller" filename="libgazebo_ros_bumper.so">
+        <plugin name="${prefix}${link_prefix}distal_gazebo_ros_tactile_controller" filename="libgazebo_ros_tactile.so">
           <alwaysOn>true</alwaysOn>
+          <robotNamespace>${ns}</robotNamespace>
           <frameName>${prefix}${link_prefix}distal</frameName>
           <updateRate>100.0</updateRate>
           <bumperTopicName>contacts/${prefix}${link_prefix}/distal</bumperTopicName>
+          <tactileTopicName>tactile_states/${prefix}${link_prefix}/distal</tactileTopicName>
         </plugin>
       </sensor>

File: sr_description/hand/xacro/tactile.ubi.xacro (robot description, xacro)
@@ -28,5 +28,5 @@
     <xacro:tactile_default_params _link="proximal"/>
     <xacro:property name="name" value="${prefix}${finger}${tactile_name}"/>
-    <sensor name="${name}" update_rate="100" group="${finger}">
+    <sensor name="${name}_sensor" update_rate="100" group="${finger}">
       <parent link="${link}" />
       <origin xyz="0 0 0" rpy="0 0 0"/>
@@ -43,5 +43,5 @@
     <xacro:tactile_default_params _link="middle"/>
     <xacro:property name="name" value="${prefix}${finger}${tactile_name}"/>
-    <sensor name="${name}" update_rate="100" group="${finger}">
+    <sensor name="${name}_sensor" update_rate="100" group="${finger}">
       <parent link="${link}" />
       <origin xyz="0 0 0" rpy="0 0 0"/>
@@ -58,5 +58,5 @@
     <xacro:property name="name" value="${prefix}${finger}${tactile_name}"/>
     <xacro:property name="tipname" value="${'thtip' if finger=='th' else 'tip'}"/>
-    <sensor name="${name}" update_rate="100" group="${finger}">
+    <sensor name="${name}_sensor" update_rate="100" group="${finger}">
       <parent link="${link}" />
       <origin xyz="0 0 0" rpy="0 0 0"/>
@@ -104,5 +104,5 @@
     <xacro:property name="mesh_scale" value="${reflect*0.00101} 0.00101 0.00101"/>
     <!-- taxels attached to lfmetacarpal -->
-    <sensor name="${prefix}lfmetacarpal" update_rate="100" group="palm">
+    <sensor name="${prefix}lfmetacarpal_sensor" update_rate="100" group="palm">
       <parent link="${link}" />
       <origin xyz="0 0 0" rpy="0 0 0"/>
@@ -116,5 +116,5 @@
     <xacro:property name="taxel_data" value="${load_yaml(taxel_dir + '/palm.taxels.ubi.yaml')}"/>
     <xacro:property name="link" value="${prefix}palm"/>
-    <sensor name="${prefix}palm" update_rate="100" group="palm">
+    <sensor name="${prefix}palm_sensor" update_rate="100" group="palm">
       <parent link="${link}" />
       <origin xyz="0 0 0" rpy="0 0 0"/>

File: sr_description/hand/xacro/thumb/thdistal.gazebo.xacro (robot description, xacro)
@@ -1,8 +1,8 @@
 <?xml version="1.0"?>
 <robot xmlns:xacro="http://www.ros.org/wiki/xacro">
-  <xacro:macro name="thdistal_gazebo" params="prefix">
+  <xacro:macro name="thdistal_gazebo" params="prefix ns:=^|''">
   <!-- prefix can be anything but usually is "r_" or  "l_" for right and left hands distinction -->
   <gazebo reference="${prefix}thdistal">
-      <sensor type="contact" name="${prefix}thdistal_contact">
+      <sensor type="contact" name="${prefix}thdistal_sensor">
         <always_on>1</always_on>
         <update_rate>1000.0</update_rate>
@@ -11,9 +11,11 @@
           <topic>${prefix}thdistal_collision</topic>
         </contact>
-        <plugin name="${prefix}thdistal_gazebo_ros_bumper_controller" filename="libgazebo_ros_bumper.so">
+        <plugin name="${prefix}thdistal_gazebo_ros_tactile_controller" filename="libgazebo_ros_tactile.so">
           <alwaysOn>true</alwaysOn>
+          <robotNamespace>${ns}</robotNamespace>
           <frameName>${prefix}thdistal</frameName>
           <updateRate>100.0</updateRate>
           <bumperTopicName>contacts/${prefix}th/distal</bumperTopicName>
+          <tactileTopicName>tactile_states/${prefix}th/distal</tactileTopicName>
         </plugin>
       </sensor>
