Commit message: added missing xacro: prefixes

File: sr_description/arm/xacro/base/shadowarm_base.urdf.xacro (robot description, xacro)
@@ -1,30 +1,30 @@
 <robot xmlns:xacro="http://www.ros.org/wiki/xacro">
-  <xacro:property name="M_PI" value="3.1415926535897931" />
-  <xacro:macro name="shadowarm_base">
-    <link name="shadowarm_base">
-      <inertial>
+<xacro:property name="M_PI" value="3.1415926535897931" />
+<xacro:macro name="shadowarm_base">
+  <link name="shadowarm_base">
+    <inertial>
         <origin xyz="0 0 0" rpy="0 0 0" />
-        <mass value="0.4" />
+      <mass value="0.4" />
         <inertia ixx="0.00071" ixy="0.0" ixz="0.0" iyy="0.00071"
         iyz="0.0" izz="0.0014" />
-      </inertial>
-      <visual>
+    </inertial>
+    <visual>
         <origin xyz="0 0 0" rpy="0 0 0" />
-        <geometry name="shadowarm_base_visual">
+      <geometry name="shadowarm_base_visual">
           <mesh filename="package://sr_description/arm/model/arm_base.dae"
           scale="0.001 0.001 0.001" />
-        </geometry>
-        <material name="LightGrey" />
-      </visual>
-      <collision>
-        <origin xyz="0 0 0.005" rpy="0 0 0" />
-        <geometry name="shadowarm_base_collision">
+      </geometry>
+      <material name="LightGrey" />
+    </visual>
+    <collision>
+      <origin xyz="0 0 0.005" rpy="0 0 0" />
+      <geometry name="shadowarm_base_collision">
           <box size="0.145 0.145 0.012" />
-        </geometry>
-      </collision>
-    </link>
-    <gazebo reference="shadowarm_base">
-      <selfCollide>false</selfCollide>
-    </gazebo>
-  </xacro:macro>
+      </geometry>
+    </collision>
+  </link>
+  <gazebo reference="shadowarm_base">
+    <selfCollide>false</selfCollide>
+  </gazebo>
+</xacro:macro>
 </robot>

File: sr_description/hand/xacro/ff_biotac_hand.urdf.xacro (robot description, xacro)
@@ -1,6 +1,6 @@
 <robot xmlns:sensor="http://playerstage.sourceforge.net/gazebo/xmlschema/#sensor"
-xmlns:controller="http://playerstage.sourceforge.net/gazebo/xmlschema/#controller"
-xmlns:interface="http://playerstage.sourceforge.net/gazebo/xmlschema/#interface"
-xmlns:xacro="http://www.ros.org/wiki/xacro">
+       xmlns:controller="http://playerstage.sourceforge.net/gazebo/xmlschema/#controller"
+       xmlns:interface="http://playerstage.sourceforge.net/gazebo/xmlschema/#interface"
+       xmlns:xacro="http://www.ros.org/wiki/xacro">
   <xacro:include filename="$(find sr_description)/hand/xacro/forearm/forearm.urdf.xacro" />
   <xacro:include filename="$(find sr_description)/hand/xacro/wrist/wrist.urdf.xacro" />
@@ -25,12 +25,12 @@
       <xacro:wrist muscletrans="${muscletrans}" prefix="${prefix}"
       reflect="${reflect}" parent="${prefix}forearm">
-        <origin xyz="0 0 0.4096" rpy="0 0 0" />
-      </xacro:wrist>
+			<origin xyz="0 0 0.4096" rpy="0 0 0" />
+			</xacro:wrist>
     </xacro:if>
-    <xacro:unless value="${muscle}">
+		<xacro:unless value="${muscle}">
       <xacro:wrist muscletrans="false" prefix="${prefix}"
       reflect="${reflect}" parent="${prefix}forearm">
-        <origin xyz="0 -0.010 0.213" rpy="0 0 0" />
-      </xacro:wrist>
+			<origin xyz="0 -0.010 0.213" rpy="0 0 0" />
+			</xacro:wrist>
     </xacro:unless>
     <!-- Palm -->

File: sr_description/hand/xacro/finger/knuckle/knuckle.urdf.xacro (robot description, xacro)
@@ -1,9 +1,9 @@
 <robot xmlns:xacro="http://www.ros.org/wiki/xacro"
-xmlns:sensor="http://playerstage.sourceforge.net/gazebo/xmlschema/#sensor"
-xmlns:controller="http://playerstage.sourceforge.net/gazebo/xmlschema/#controller"
-xmlns:joint="http://playerstage.sourceforge.net/gazebo/xmlschema/#slider"
-xmlns:interface="http://playerstage.sourceforge.net/gazebo/xmlschema/#interface"
-xmlns:body="http://playerstage.sourceforge.net/gazebo/xmlschema/#body"
-xmlns:geom="http://playerstage.sourceforge.net/gazebo/xmlschema/#geom">
+       xmlns:sensor="http://playerstage.sourceforge.net/gazebo/xmlschema/#sensor"
+       xmlns:controller="http://playerstage.sourceforge.net/gazebo/xmlschema/#controller"
+       xmlns:joint="http://playerstage.sourceforge.net/gazebo/xmlschema/#slider"
+       xmlns:interface="http://playerstage.sourceforge.net/gazebo/xmlschema/#interface"
+       xmlns:body="http://playerstage.sourceforge.net/gazebo/xmlschema/#body"
+       xmlns:geom="http://playerstage.sourceforge.net/gazebo/xmlschema/#geom">
   <xacro:include filename="$(find sr_description)/hand/xacro/finger/knuckle/knuckle.gazebo.xacro" />
   <xacro:include filename="$(find sr_description)/hand/xacro/finger/knuckle/knuckle.transmission.xacro" />
@@ -18,4 +18,5 @@
       <inertial>
         <origin xyz="0 0 0" rpy="0 0 0" />
+        <!--<insert_block name="origin" /> -->
         <mass value="0.008" />
         <inertia ixx="0.00000026" ixy="0.0" ixz="0.0"

File: sr_description/hand/xacro/forearm/forearm_lite.urdf.xacro (robot description, xacro)
@@ -3,41 +3,42 @@
   <!-- prefix can be anything but usually is "r_" or  "l_" for right and left hands distinction -->
   <xacro:macro name="forearm" params="muscle prefix">
-    <link name="${prefix}forearm">
-      <inertial>
+      <property name="M_PI" value="3.1415926535897931" />
+      <link name="${prefix}forearm">
+        <inertial>
         <origin xyz="0 0 0.09" rpy="0 0 0" />
-        <!-- TODO: This is a rough estimate. Total hand is 2359g -->
-        <mass value="1.8" />
+          <!-- TODO: This is a rough estimate. Total hand is 2359g -->
+          <mass value="1.8" />
         <inertia ixx="0.108" ixy="0.0" ixz="0.0" iyy="0.108"
         iyz="0.0" izz="0.054" />
-      </inertial>
-      <visual>
-        <origin xyz="0 0 0" rpy="0 0 ${M_PI/2}" />
-        <geometry name="${prefix}forearm_visual">
+        </inertial>
+        <visual>
+          <origin xyz="0 0 0" rpy="0 0 ${M_PI/2}" />
+          <geometry name="${prefix}forearm_visual">
+            <xacro:if value="${muscle}">
+               <mesh filename="package://sr_description/hand/model/forearm_lite.dae"
+            scale="1.0 1.0 1.0" />
+            </xacro:if>
+            <xacro:unless value="${muscle}">
+               <mesh filename="package://sr_description/hand/model/forearm_lite.dae"
+            scale="1.0 1.0 1.0" />
+            </xacro:unless>
+          </geometry>
+          <material name="Grey" />
+        </visual>
+        <collision>
           <xacro:if value="${muscle}">
-            <mesh filename="package://sr_description/hand/model/forearm_lite.dae"
-            scale="1.0 1.0 1.0" />
-          </xacro:if>
+            <origin xyz="0 0 0.185" rpy="0 0 0" />
+            <geometry name="${prefix}forearm_collision">
+            <cylinder radius="0.075" length="0.37" />
+            </geometry>
+        </xacro:if>
           <xacro:unless value="${muscle}">
-            <mesh filename="package://sr_description/hand/model/forearm_lite.dae"
-            scale="1.0 1.0 1.0" />
+            <origin xyz="0 0 0.0775" rpy="0 0 0" />
+            <geometry name="${prefix}forearm_collision">
+              <box size="0.109 0.120 0.155" />
+            </geometry>
           </xacro:unless>
-        </geometry>
-        <material name="Grey" />
-      </visual>
-      <collision>
-        <xacro:if value="${muscle}">
-          <origin xyz="0 0 0.185" rpy="0 0 0" />
-          <geometry name="${prefix}forearm_collision">
-            <cylinder radius="0.075" length="0.37" />
-          </geometry>
-        </xacro:if>
-        <xacro:unless value="${muscle}">
-          <origin xyz="0 0 0.0775" rpy="0 0 0" />
-          <geometry name="${prefix}forearm_collision">
-            <box size="0.109 0.120 0.155" />
-          </geometry>
-        </xacro:unless>
-      </collision>
-    </link>
+        </collision>
+      </link>
   </xacro:macro>
 </robot>

File: sr_description/hand/xacro/full_hand.urdf.xacro (robot description, xacro)
@@ -1,6 +1,6 @@
 <robot xmlns:sensor="http://playerstage.sourceforge.net/gazebo/xmlschema/#sensor"
-xmlns:controller="http://playerstage.sourceforge.net/gazebo/xmlschema/#controller"
-xmlns:interface="http://playerstage.sourceforge.net/gazebo/xmlschema/#interface"
-xmlns:xacro="http://www.ros.org/wiki/xacro">
+       xmlns:controller="http://playerstage.sourceforge.net/gazebo/xmlschema/#controller"
+       xmlns:interface="http://playerstage.sourceforge.net/gazebo/xmlschema/#interface"
+       xmlns:xacro="http://www.ros.org/wiki/xacro">
   <xacro:include filename="$(find sr_description)/hand/xacro/forearm/forearm.urdf.xacro" />
   <xacro:include filename="$(find sr_description)/hand/xacro/wrist/wrist.urdf.xacro" />
@@ -22,15 +22,15 @@
     <xacro:forearm muscle="${muscle}" prefix="${prefix}" />
     <!-- Wrist -->
-    <xacro:if value="${muscle}">
+		<xacro:if value="${muscle}">
       <xacro:wrist muscletrans="${muscletrans}" prefix="${prefix}"
       reflect="${reflect}" parent="${prefix}forearm">
-        <origin xyz="0 0 0.4096" rpy="0 0 0" />
-      </xacro:wrist>
+			<origin xyz="0 0 0.4096" rpy="0 0 0" />
+			</xacro:wrist>
     </xacro:if>
-    <xacro:unless value="${muscle}">
+		<xacro:unless value="${muscle}">
       <xacro:wrist muscletrans="false" prefix="${prefix}"
       reflect="${reflect}" parent="${prefix}forearm">
-        <origin xyz="0 -0.010 0.213" rpy="0 0 0" />
-      </xacro:wrist>
+			<origin xyz="0 -0.010 0.213" rpy="0 0 0" />
+			</xacro:wrist>
     </xacro:unless>
     <!-- Palm -->

File: sr_description/hand/xacro/hand_lite.urdf.xacro (robot description, xacro)
@@ -1,6 +1,6 @@
 <robot xmlns:sensor="http://playerstage.sourceforge.net/gazebo/xmlschema/#sensor"
-xmlns:controller="http://playerstage.sourceforge.net/gazebo/xmlschema/#controller"
-xmlns:interface="http://playerstage.sourceforge.net/gazebo/xmlschema/#interface"
-xmlns:xacro="http://www.ros.org/wiki/xacro">
+       xmlns:controller="http://playerstage.sourceforge.net/gazebo/xmlschema/#controller"
+       xmlns:interface="http://playerstage.sourceforge.net/gazebo/xmlschema/#interface"
+       xmlns:xacro="http://www.ros.org/wiki/xacro">
   <xacro:include filename="$(find sr_description)/hand/xacro/forearm/forearm_lite.urdf.xacro" />
   <xacro:include filename="$(find sr_description)/hand/xacro/wrist/wrist.urdf.xacro" />
@@ -46,7 +46,7 @@
 		    reflect="${reflect}" link_prefix="mf" joint_prefix="MF"
 		    parent="${prefix}palm">
-	<origin xyz="${reflect*0.011} 0 0.099" rpy="0 0 0" />
-	<axis xyz="0 ${-1*reflect} 0" />
-      </xacro:finger>
+      <origin xyz="${reflect*0.011} 0 0.099" rpy="0 0 0" />
+      <axis xyz="0 ${-1*reflect} 0" />
+    </xacro:finger>
     </xacro:unless>
     <!-- Ring Finger -->

File: sr_description/hand/xacro/one_finger_unit.urdf.xacro (robot description, xacro)
@@ -1,6 +1,6 @@
 <robot xmlns:sensor="http://playerstage.sourceforge.net/gazebo/xmlschema/#sensor"
-xmlns:controller="http://playerstage.sourceforge.net/gazebo/xmlschema/#controller"
-xmlns:interface="http://playerstage.sourceforge.net/gazebo/xmlschema/#interface"
-xmlns:xacro="http://www.ros.org/wiki/xacro">
+       xmlns:controller="http://playerstage.sourceforge.net/gazebo/xmlschema/#controller"
+       xmlns:interface="http://playerstage.sourceforge.net/gazebo/xmlschema/#interface"
+       xmlns:xacro="http://www.ros.org/wiki/xacro">
   <xacro:include filename="$(find sr_description)/hand/xacro/forearm/forearm.urdf.xacro" />
   <xacro:include filename="$(find sr_description)/hand/xacro/finger/fingers.urdf.xacro" />
@@ -19,23 +19,23 @@
     <xacro:forearm muscle="${muscle}" prefix="${prefix}" />
     <!-- Dummy Palm -->
-    <link name="${prefix}dummy_palm">
+		<link name="${prefix}dummy_palm">
       <inertial>
-        <mass value="0.010" />
-        <origin xyz="0 0 0" />
+				<mass value="0.010" />
+				<origin xyz="0 0 0" />
         <inertia ixx="1.0" ixy="0.0" ixz="0.0" iyy="0.0" iyz="0.0"
-        izz="0.0" />
+				izz="0.0" />
       </inertial>
       <visual>
-        <origin xyz="0 0 0.0505" rpy="0 0 0" />
-        <geometry name="${prefix}dummy_palm_visual">
-          <box size="0.015 0.015 0.110" />
-        </geometry>
-        <material name="Grey" />
+				<origin xyz="0 0 0.0505" rpy="0 0 0" />
+				<geometry name="${prefix}dummy_palm_visual">
+					<box size="0.015 0.015 0.110" />
+				</geometry>
+				<material name="Grey" />
       </visual>
       <collision>
-        <origin xyz="0 0 0.0" rpy="0 0 0" />
-        <geometry name="${prefix}dummy_palm_collision_geom">
-          <box size="0.015 0.015 0.110" />
-        </geometry>
+				<origin xyz="0 0 0.0" rpy="0 0 0" />
+				<geometry name="${prefix}dummy_palm_collision_geom">
+					<box size="0.015 0.015 0.110" />
+				</geometry>
       </collision>
     </link>

File: sr_description/hand/xacro/th_ff_rf_ellipsoid_hand.urdf.xacro (robot description, xacro)
@@ -1,6 +1,6 @@
 <robot xmlns:sensor="http://playerstage.sourceforge.net/gazebo/xmlschema/#sensor"
-xmlns:controller="http://playerstage.sourceforge.net/gazebo/xmlschema/#controller"
-xmlns:interface="http://playerstage.sourceforge.net/gazebo/xmlschema/#interface"
-xmlns:xacro="http://www.ros.org/wiki/xacro">
+       xmlns:controller="http://playerstage.sourceforge.net/gazebo/xmlschema/#controller"
+       xmlns:interface="http://playerstage.sourceforge.net/gazebo/xmlschema/#interface"
+       xmlns:xacro="http://www.ros.org/wiki/xacro">
   <xacro:include filename="$(find sr_description)/hand/xacro/forearm/forearm.urdf.xacro" />
   <xacro:include filename="$(find sr_description)/hand/xacro/wrist/wrist.urdf.xacro" />
@@ -25,12 +25,12 @@
       <xacro:wrist muscletrans="${muscletrans}" prefix="${prefix}"
       reflect="${reflect}" parent="${prefix}forearm">
-        <origin xyz="0 0 0.4096" rpy="0 0 0" />
-      </xacro:wrist>
+			<origin xyz="0 0 0.4096" rpy="0 0 0" />
+			</xacro:wrist>
     </xacro:if>
-    <xacro:unless value="${muscle}">
+		<xacro:unless value="${muscle}">
       <xacro:wrist muscletrans="false" prefix="${prefix}"
       reflect="${reflect}" parent="${prefix}forearm">
-        <origin xyz="0 -0.010 0.213" rpy="0 0 0" />
-      </xacro:wrist>
+			<origin xyz="0 -0.010 0.213" rpy="0 0 0" />
+			</xacro:wrist>
     </xacro:unless>
     <!-- Palm -->

File: sr_description/hand/xacro/three_biotac_fingers_hand.urdf.xacro (robot description, xacro)
@@ -1,6 +1,6 @@
 <robot xmlns:sensor="http://playerstage.sourceforge.net/gazebo/xmlschema/#sensor"
-xmlns:controller="http://playerstage.sourceforge.net/gazebo/xmlschema/#controller"
-xmlns:interface="http://playerstage.sourceforge.net/gazebo/xmlschema/#interface"
-xmlns:xacro="http://www.ros.org/wiki/xacro">
+       xmlns:controller="http://playerstage.sourceforge.net/gazebo/xmlschema/#controller"
+       xmlns:interface="http://playerstage.sourceforge.net/gazebo/xmlschema/#interface"
+       xmlns:xacro="http://www.ros.org/wiki/xacro">
   <xacro:include filename="$(find sr_description)/hand/xacro/forearm/forearm.urdf.xacro" />
   <xacro:include filename="$(find sr_description)/hand/xacro/wrist/wrist.urdf.xacro" />
@@ -25,12 +25,12 @@
       <xacro:wrist muscletrans="${muscletrans}" prefix="${prefix}"
       reflect="${reflect}" parent="${prefix}forearm">
-        <origin xyz="0 0 0.4096" rpy="0 0 0" />
-      </xacro:wrist>
+			<origin xyz="0 0 0.4096" rpy="0 0 0" />
+			</xacro:wrist>
     </xacro:if>
-    <xacro:unless value="${muscle}">
+		<xacro:unless value="${muscle}">
       <xacro:wrist muscletrans="false" prefix="${prefix}"
       reflect="${reflect}" parent="${prefix}forearm">
-        <origin xyz="0 -0.010 0.213" rpy="0 0 0" />
-      </xacro:wrist>
+			<origin xyz="0 -0.010 0.213" rpy="0 0 0" />
+			</xacro:wrist>
     </xacro:unless>
     <!-- Palm -->

File: sr_description/hand/xacro/three_fingers_hand.urdf.xacro (robot description, xacro)
@@ -1,6 +1,6 @@
 <robot xmlns:sensor="http://playerstage.sourceforge.net/gazebo/xmlschema/#sensor"
-xmlns:controller="http://playerstage.sourceforge.net/gazebo/xmlschema/#controller"
-xmlns:interface="http://playerstage.sourceforge.net/gazebo/xmlschema/#interface"
-xmlns:xacro="http://www.ros.org/wiki/xacro">
+       xmlns:controller="http://playerstage.sourceforge.net/gazebo/xmlschema/#controller"
+       xmlns:interface="http://playerstage.sourceforge.net/gazebo/xmlschema/#interface"
+       xmlns:xacro="http://www.ros.org/wiki/xacro">
   <xacro:include filename="$(find sr_description)/hand/xacro/forearm/forearm.urdf.xacro" />
   <xacro:include filename="$(find sr_description)/hand/xacro/wrist/wrist.urdf.xacro" />

File: sr_description/hand/xacro/wrist/wrist.urdf.xacro (robot description, xacro)
@@ -9,16 +9,16 @@
     <link name="${prefix}wrist">
       <inertial>
-        <origin xyz="0 0 0.029" rpy="0 0 0" />
-        <mass value="0.1" />
+		  <origin xyz="0 0 0.029" rpy="0 0 0" />
+		  <mass value="0.1" />
         <inertia ixx="0.000035" ixy="0.0" ixz="0.0" iyy="0.000064"
         iyz="0.0" izz="0.0000438" />
       </inertial>
       <visual>
-        <origin xyz="0 0 0" rpy="0 0 0" />
-        <geometry name="${prefix}wrist_visual">
+		  <origin xyz="0 0 0" rpy="0 0 0" />
+		  <geometry name="${prefix}wrist_visual">
           <mesh filename="package://sr_description/hand/model/wrist.dae"
-          scale="${reflect*0.001} 0.001 0.001" />
-        </geometry>
-        <material name="LightGrey" />
+					 scale="${reflect*0.001} 0.001 0.001" />
+		  </geometry>
+		  <material name="LightGrey" />
       </visual>
       <collision>

File: sr_description/other/xacro/kinect/shadowarm_kinect.urdf.xacro (robot description, xacro)
@@ -5,7 +5,7 @@
     <joint name="base_camera_joint" type="fixed">
       <!--        <origin xyz="0.00724 0.153 0.4405"
-          rpy="-${M_PI/2} 0.5236 -0.2618" /> -->
+	  rpy="-${M_PI/2} 0.5236 -0.2618" /> -->
       <origin xyz="0.01216 0.1713 0.433"
-      rpy="-${M_PI/2} ${M_PI/4} -${M_PI/12}" />
+	      rpy="-${M_PI/2} ${M_PI/4} -${M_PI/12}" />
       <parent link="${parent}" />
       <child link="camera_link" />
@@ -13,6 +13,6 @@
     <link name="camera_link">
       <inertial>
-        <mass value="0.01" />
-        <origin xyz="0 0 0" />
+	<mass value="0.01" />
+	<origin xyz="0 0 0" />
         <inertia ixx="0.001" ixy="0.0" ixz="0.0" iyy="0.001"
         iyz="0.0" izz="0.001" />
@@ -20,13 +20,13 @@
       <visual>
         <origin xyz=" 0 0 0" rpy="0 0 0" />
-        <geometry>
+	<geometry>
           <mesh filename="package://sr_description/other/model/kinect.dae" />
-        </geometry>
+	</geometry>
       </visual>
       <collision>
-        <origin xyz="0.0 0.0 0.0" rpy="0 0 0" />
-        <geometry>
+	<origin xyz="0.0 0.0 0.0" rpy="0 0 0" />
+	<geometry>
           <box size="0.0730 .2760 0.0720" />
-        </geometry>
+	</geometry>
       </collision>
     </link>
@@ -38,6 +38,6 @@
     <link name="camera_depth_frame">
       <inertial>
-        <mass value="0.01" />
-        <origin xyz="0 0 0" />
+	<mass value="0.01" />
+	<origin xyz="0 0 0" />
         <inertia ixx="0.001" ixy="0.0" ixz="0.0" iyy="0.001"
         iyz="0.0" izz="0.001" />
@@ -51,6 +51,6 @@
     <link name="camera_depth_optical_frame">
       <inertial>
-        <mass value="0.001" />
-        <origin xyz="0 0 0" />
+	<mass value="0.001" />
+	<origin xyz="0 0 0" />
         <inertia ixx="0.0001" ixy="0.0" ixz="0.0" iyy="0.0001"
         iyz="0.0" izz="0.0001" />
@@ -64,6 +64,6 @@
     <link name="camera_rgb_frame">
       <inertial>
-        <mass value="0.001" />
-        <origin xyz="0 0 0" />
+	<mass value="0.001" />
+	<origin xyz="0 0 0" />
         <inertia ixx="0.0001" ixy="0.0" ixz="0.0" iyy="0.0001"
         iyz="0.0" izz="0.0001" />
@@ -77,6 +77,6 @@
     <link name="camera_rgb_optical_frame">
       <inertial>
-        <mass value="0.001" />
-        <origin xyz="0 0 0" />
+	<mass value="0.001" />
+	<origin xyz="0 0 0" />
         <inertia ixx="0.0001" ixy="0.0" ixz="0.0" iyy="0.0001"
         iyz="0.0" izz="0.0001" />
