Commit message: added missing xacro: prefixes

File: sr_description/hand/xacro/forearm/forearm_lite.urdf.xacro (robot description, xacro)
@@ -3,32 +3,33 @@
   <!-- prefix can be anything but usually is "r_" or  "l_" for right and left hands distinction -->
   <xacro:macro name="forearm" params="muscle prefix">
-    <link name="${prefix}forearm">
-      <inertial>
+      <property name="M_PI" value="3.1415926535897931" />
+      <link name="${prefix}forearm">
+        <inertial>
         <origin xyz="0 0 0.09" rpy="0 0 0" />
-        <!-- TODO: This is a rough estimate. Total hand is 2359g -->
-        <mass value="1.8" />
+          <!-- TODO: This is a rough estimate. Total hand is 2359g -->
+          <mass value="1.8" />
         <inertia ixx="0.108" ixy="0.0" ixz="0.0" iyy="0.108"
         iyz="0.0" izz="0.054" />
-      </inertial>
-      <visual>
-        <origin xyz="0 0 0" rpy="0 0 ${M_PI/2}" />
-        <geometry name="${prefix}forearm_visual">
+        </inertial>
+        <visual>
+          <origin xyz="0 0 0" rpy="0 0 ${M_PI/2}" />
+          <geometry name="${prefix}forearm_visual">
+            <xacro:if value="${muscle}">
+               <mesh filename="package://sr_description/hand/model/forearm_lite.dae"
+            scale="1.0 1.0 1.0" />
+            </xacro:if>
+            <xacro:unless value="${muscle}">
+               <mesh filename="package://sr_description/hand/model/forearm_lite.dae"
+            scale="1.0 1.0 1.0" />
+            </xacro:unless>
+          </geometry>
+          <material name="Grey" />
+        </visual>
+        <collision>
           <xacro:if value="${muscle}">
-            <mesh filename="package://sr_description/hand/model/forearm_lite.dae"
-            scale="1.0 1.0 1.0" />
-          </xacro:if>
-          <xacro:unless value="${muscle}">
-            <mesh filename="package://sr_description/hand/model/forearm_lite.dae"
-            scale="1.0 1.0 1.0" />
-          </xacro:unless>
-        </geometry>
-        <material name="Grey" />
-      </visual>
-      <collision>
-        <xacro:if value="${muscle}">
-          <origin xyz="0 0 0.185" rpy="0 0 0" />
-          <geometry name="${prefix}forearm_collision">
+            <origin xyz="0 0 0.185" rpy="0 0 0" />
+            <geometry name="${prefix}forearm_collision">
             <cylinder radius="0.075" length="0.37" />
-          </geometry>
+            </geometry>
         </xacro:if>
         <xacro:unless value="${muscle}">

File: sr_description/hand/xacro/one_finger_unit.urdf.xacro (robot description, xacro)
@@ -1,6 +1,6 @@
 <robot xmlns:sensor="http://playerstage.sourceforge.net/gazebo/xmlschema/#sensor"
-xmlns:controller="http://playerstage.sourceforge.net/gazebo/xmlschema/#controller"
-xmlns:interface="http://playerstage.sourceforge.net/gazebo/xmlschema/#interface"
-xmlns:xacro="http://www.ros.org/wiki/xacro">
+       xmlns:controller="http://playerstage.sourceforge.net/gazebo/xmlschema/#controller"
+       xmlns:interface="http://playerstage.sourceforge.net/gazebo/xmlschema/#interface"
+       xmlns:xacro="http://www.ros.org/wiki/xacro">
   <xacro:include filename="$(find sr_description)/hand/xacro/forearm/forearm.urdf.xacro" />
   <xacro:include filename="$(find sr_description)/hand/xacro/finger/fingers.urdf.xacro" />
@@ -24,5 +24,5 @@
         <origin xyz="0 0 0" />
         <inertia ixx="1.0" ixy="0.0" ixz="0.0" iyy="0.0" iyz="0.0"
-        izz="0.0" />
+                 izz="0.0" />
       </inertial>
       <visual>
