Commit message: Changed the forearm collision model to cylinder again and attached hand to world Fixed rviz in test to match new prefix and use world as ref frame

File: sr_description/hand/xacro/forearm/forearm.urdf.xacro (robot description, xacro)
@@ -34,5 +34,6 @@
           <origin xyz="0 0 0.092" rpy="0 0 0" />
           <geometry name="${prefix}forearm_collision">
-            <box size="0.140 0.140 0.184" />
+            <cylinder radius="0.07" length="0.184"/>
+            <!--<box size="0.140 0.140 0.184" />-->
           </geometry>
         </xacro:unless>

File: sr_description/robots/shadowhand_edc_muscle.urdf.xacro (robot description, xacro)
@@ -7,4 +7,11 @@
   <xacro:include filename="$(find sr_description)/hand/xacro/full_hand.urdf.xacro" />
   <xacro:include filename="$(find sr_description)/other/xacro/gazebo/gazebo.urdf.xacro" />
+  <!-- hand with cylindrical base drifts in gazebo, attach it to the world -->
+  <link name="world" />
+  <joint name="rh_world_joint" type="fixed">
+    <parent link="world" />
+    <child link="rh_forearm_disk" />
+    <origin xyz="0.0 0.0 0.0" rpy="0.0 0.0 0.0" />
+  </joint>
   <xacro:shadowhand muscletrans="true" muscle="true" bio="false" bt_sp="false"
   ubi="false" eli="false" reflect="1.0" prefix="rh_" />

File: sr_description/robots/shadowhand_edc_muscle_biotac.urdf.xacro (robot description, xacro)
@@ -7,4 +7,11 @@
   <xacro:include filename="$(find sr_description)/hand/xacro/full_hand.urdf.xacro" />
   <xacro:include filename="$(find sr_description)/other/xacro/gazebo/gazebo.urdf.xacro" />
+  <!-- hand with cylindrical base drifts in gazebo, attach it to the world -->
+  <link name="world" />
+  <joint name="rh_world_joint" type="fixed">
+    <parent link="world" />
+    <child link="rh_forearm_disk" />
+    <origin xyz="0.0 0.0 0.0" rpy="0.0 0.0 0.0" />
+  </joint>
   <!-- C6 hand with BioTAC sensor
   (C) 2012 fnh, hendrich@informatik.uni-hamburg.de

File: sr_description/robots/shadowhand_left_edc_muscle.urdf.xacro (robot description, xacro)
@@ -7,4 +7,11 @@
   <xacro:include filename="$(find sr_description)/hand/xacro/full_hand.urdf.xacro" />
   <xacro:include filename="$(find sr_description)/other/xacro/gazebo/gazebo.urdf.xacro" />
+  <!-- hand with cylindrical base drifts in gazebo, attach it to the world -->
+  <link name="world" />
+  <joint name="lh_world_joint" type="fixed">
+    <parent link="world" />
+    <child link="lh_forearm_disk" />
+    <origin xyz="0.0 0.0 0.0" rpy="0.0 0.0 0.0" />
+  </joint>
   <xacro:shadowhand muscletrans="true" muscle="true" bio="false" bt_sp="false"
   ubi="false" eli="false" reflect="-1.0" prefix="lh_" />

File: sr_description/robots/shadowhand_left_motor.urdf.xacro (robot description, xacro)
@@ -7,4 +7,11 @@
   <xacro:include filename="$(find sr_description)/hand/xacro/full_hand.urdf.xacro" />
   <xacro:include filename="$(find sr_description)/other/xacro/gazebo/gazebo.urdf.xacro" />
+  <!-- hand with cylindrical base drifts in gazebo, attach it to the world -->
+  <link name="world" />
+  <joint name="lh_world_joint" type="fixed">
+    <parent link="world" />
+    <child link="lh_forearm" />
+    <origin xyz="0.0 0.0 0.0" rpy="0.0 0.0 0.0" />
+  </joint>
   <xacro:shadowhand muscletrans="false" muscle="false" bio="false" bt_sp="false"
   ubi="false" eli="false" reflect="-1.0" prefix="lh_" />

File: sr_description/robots/shadowhand_left_motor_biotac.urdf.xacro (robot description, xacro)
@@ -7,4 +7,11 @@
   <xacro:include filename="$(find sr_description)/hand/xacro/full_hand.urdf.xacro" />
   <xacro:include filename="$(find sr_description)/other/xacro/gazebo/gazebo.urdf.xacro" />
+  <!-- hand with cylindrical base drifts in gazebo, attach it to the world -->
+  <link name="world" />
+  <joint name="lh_world_joint" type="fixed">
+    <parent link="world" />
+    <child link="lh_forearm" />
+    <origin xyz="0.0 0.0 0.0" rpy="0.0 0.0 0.0" />
+  </joint>
   <xacro:shadowhand muscletrans="false" muscle="false" bio="true" bt_sp="false"
   ubi="false" eli="false" reflect="-1.0" prefix="lh_" />

File: sr_description/robots/shadowhand_left_muscle.urdf.xacro (robot description, xacro)
@@ -7,4 +7,11 @@
   <xacro:include filename="$(find sr_description)/hand/xacro/full_hand.urdf.xacro" />
   <xacro:include filename="$(find sr_description)/other/xacro/gazebo/gazebo.urdf.xacro" />
+  <!-- hand with cylindrical base drifts in gazebo, attach it to the world -->
+  <link name="world" />
+  <joint name="lh_world_joint" type="fixed">
+    <parent link="world" />
+    <child link="lh_forearm_disk" />
+    <origin xyz="0.0 0.0 0.0" rpy="0.0 0.0 0.0" />
+  </joint>
   <xacro:shadowhand muscletrans="false" muscle="true" bio="false" bt_sp="false"
   ubi="false" eli="false" reflect="-1.0" prefix="lh_" />

File: sr_description/robots/shadowhand_motor.urdf.xacro (robot description, xacro)
@@ -7,4 +7,11 @@
     <xacro:include filename="$(find sr_description)/hand/xacro/full_hand.urdf.xacro"/>
     <xacro:include filename="$(find sr_description)/other/xacro/gazebo/gazebo.urdf.xacro"/>
+    <!-- hand with cylindrical base drifts in gazebo, attach it to the world -->
+    <link name="world" />
+    <joint name="rh_world_joint" type="fixed">
+      <parent link="world" />
+      <child link="rh_forearm" />
+      <origin xyz="0.0 0.0 0.0" rpy="0.0 0.0 0.0" />
+    </joint>
     <xacro:shadowhand muscletrans="false" muscle="false" bio="false" bt_sp="false"
                       ubi="false" eli="false" reflect="1.0" prefix="rh_"/>

File: sr_description/robots/shadowhand_motor_biotac.urdf.xacro (robot description, xacro)
@@ -7,4 +7,11 @@
   <xacro:include filename="$(find sr_description)/hand/xacro/full_hand.urdf.xacro" />
   <xacro:include filename="$(find sr_description)/other/xacro/gazebo/gazebo.urdf.xacro" />
+  <!-- hand with cylindrical base drifts in gazebo, attach it to the world -->
+  <link name="world" />
+  <joint name="rh_world_joint" type="fixed">
+    <parent link="world" />
+    <child link="rh_forearm" />
+    <origin xyz="0.0 0.0 0.0" rpy="0.0 0.0 0.0" />
+  </joint>
   <!-- C6 hand with BioTAC sensor
   (C) 2012 fnh, hendrich@informatik.uni-hamburg.de

File: sr_description/robots/shadowhand_motor_btsp.urdf.xacro (robot description, xacro)
@@ -7,4 +7,11 @@
   <xacro:include filename="$(find sr_description)/hand/xacro/full_hand.urdf.xacro" />
   <xacro:include filename="$(find sr_description)/other/xacro/gazebo/gazebo.urdf.xacro" />
+  <!-- hand with cylindrical base drifts in gazebo, attach it to the world -->
+  <link name="world" />
+  <joint name="rh_world_joint" type="fixed">
+    <parent link="world" />
+    <child link="rh_forearm" />
+    <origin xyz="0.0 0.0 0.0" rpy="0.0 0.0 0.0" />
+  </joint>
   <xacro:shadowhand muscletrans="false" muscle="false" bio="false" bt_sp="true"
   ubi="false" eli="false" reflect="1.0" prefix="rh_" />

File: sr_description/robots/shadowhand_motor_ellipsoid.urdf.xacro (robot description, xacro)
@@ -7,4 +7,11 @@
   <xacro:include filename="$(find sr_description)/hand/xacro/full_hand.urdf.xacro" />
   <xacro:include filename="$(find sr_description)/other/xacro/gazebo/gazebo.urdf.xacro" />
+  <!-- hand with cylindrical base drifts in gazebo, attach it to the world -->
+  <link name="world" />
+  <joint name="rh_world_joint" type="fixed">
+    <parent link="world" />
+    <child link="rh_forearm" />
+    <origin xyz="0.0 0.0 0.0" rpy="0.0 0.0 0.0" />
+  </joint>
   <xacro:shadowhand muscletrans="false" muscle="false" bio="false" bt_sp="false"
   ubi="false" eli="true" reflect="1.0" prefix="rh_" />

File: sr_description/robots/shadowhand_motor_ff_biotac.urdf.xacro (robot description, xacro)
@@ -7,4 +7,11 @@
   <xacro:include filename="$(find sr_description)/hand/xacro/ff_biotac_hand.urdf.xacro" />
   <xacro:include filename="$(find sr_description)/other/xacro/gazebo/gazebo.urdf.xacro" />
+  <!-- hand with cylindrical base drifts in gazebo, attach it to the world -->
+  <link name="world" />
+  <joint name="rh_world_joint" type="fixed">
+    <parent link="world" />
+    <child link="rh_forearm" />
+    <origin xyz="0.0 0.0 0.0" rpy="0.0 0.0 0.0" />
+  </joint>
   <!-- bio is used for all other fingers since ff is forced at bio -->
   <xacro:shadowhand muscletrans="false" muscle="false" bio="false" bt_sp="false"

File: sr_description/robots/shadowhand_motor_th_ff_rf_ellipsoid.urdf.xacro (robot description, xacro)
@@ -7,4 +7,11 @@
   <xacro:include filename="$(find sr_description)/hand/xacro/th_ff_rf_ellipsoid_hand.urdf.xacro" />
   <xacro:include filename="$(find sr_description)/other/xacro/gazebo/gazebo.urdf.xacro" />
+  <!-- hand with cylindrical base drifts in gazebo, attach it to the world -->
+  <link name="world" />
+  <joint name="rh_world_joint" type="fixed">
+    <parent link="world" />
+    <child link="rh_forearm" />
+    <origin xyz="0.0 0.0 0.0" rpy="0.0 0.0 0.0" />
+  </joint>
   <!-- eli is used for other fingers since th, ff and rf are forced to eli -->
   <xacro:shadowhand muscletrans="false" muscle="false" bio="false" bt_sp="false"

File: sr_description/robots/shadowhand_muscle.urdf.xacro (robot description, xacro)
@@ -7,4 +7,11 @@
   <xacro:include filename="$(find sr_description)/hand/xacro/full_hand.urdf.xacro" />
   <xacro:include filename="$(find sr_description)/other/xacro/gazebo/gazebo.urdf.xacro" />
+  <!-- hand with cylindrical base drifts in gazebo, attach it to the world -->
+  <link name="world" />
+  <joint name="rh_world_joint" type="fixed">
+    <parent link="world" />
+    <child link="rh_forearm_disk" />
+    <origin xyz="0.0 0.0 0.0" rpy="0.0 0.0 0.0" />
+  </joint>
   <xacro:shadowhand muscletrans="false" muscle="true" bio="false" bt_sp="false"
   ubi="false" eli="false" reflect="1.0" prefix="rh_" />

File: sr_description/robots/shadowhand_muscle_biotac.urdf.xacro (robot description, xacro)
@@ -10,4 +10,11 @@
   (C) 2012 fnh, hendrich@informatik.uni-hamburg.de
 -->
+  <!-- hand with cylindrical base drifts in gazebo, attach it to the world -->
+  <link name="world" />
+  <joint name="rh_world_joint" type="fixed">
+    <parent link="world" />
+    <child link="rh_forearm_disk" />
+    <origin xyz="0.0 0.0 0.0" rpy="0.0 0.0 0.0" />
+  </joint>
   <xacro:shadowhand muscletrans="false" muscle="true" bio="true" bt_sp="false"
   ubi="false" eli="false" reflect="1.0" prefix="rh_" />

File: sr_description/robots/sr_one_finger_motor.urdf.xacro (robot description, xacro)
@@ -7,4 +7,11 @@
   <xacro:include filename="$(find sr_description)/hand/xacro/one_finger_unit.urdf.xacro" />
   <xacro:include filename="$(find sr_description)/other/xacro/gazebo/gazebo.urdf.xacro" />
+  <!-- hand with cylindrical base drifts in gazebo, attach it to the world -->
+  <link name="world" />
+  <joint name="rh_world_joint" type="fixed">
+    <parent link="world" />
+    <child link="rh_forearm" />
+    <origin xyz="0.0 0.0 0.0" rpy="0.0 0.0 0.0" />
+  </joint>
   <xacro:shadowhand muscletrans="false" muscle="false" bio="false" bt_sp="false"
   ubi="false" eli="false" reflect="1.0" prefix="rh_" />

File: sr_description/robots/sr_three_finger_edc_muscle_biotac.urdf.xacro (robot description, xacro)
@@ -7,4 +7,11 @@
   <xacro:include filename="$(find sr_description)/hand/xacro/three_fingers_hand.urdf.xacro" />
   <xacro:include filename="$(find sr_description)/other/xacro/gazebo/gazebo.urdf.xacro" />
+  <!-- hand with cylindrical base drifts in gazebo, attach it to the world -->
+  <link name="world" />
+  <joint name="rh_world_joint" type="fixed">
+    <parent link="world" />
+    <child link="rh_forearm" />
+    <origin xyz="0.0 0.0 0.0" rpy="0.0 0.0 0.0" />
+  </joint>
   <xacro:shadowhand muscletrans="true" muscle="true" bio="true" bt_sp="false"
   ubi="false" eli="false" reflect="1.0" prefix="rh_" />

File: sr_description/robots/sr_three_finger_motor.urdf.xacro (robot description, xacro)
@@ -7,4 +7,11 @@
   <xacro:include filename="$(find sr_description)/hand/xacro/three_fingers_hand.urdf.xacro" />
   <xacro:include filename="$(find sr_description)/other/xacro/gazebo/gazebo.urdf.xacro" />
+  <!-- hand with cylindrical base drifts in gazebo, attach it to the world -->
+  <link name="world" />
+  <joint name="rh_world_joint" type="fixed">
+    <parent link="world" />
+    <child link="rh_forearm" />
+    <origin xyz="0.0 0.0 0.0" rpy="0.0 0.0 0.0" />
+  </joint>
   <xacro:shadowhand muscletrans="false" muscle="false" bio="false" bt_sp="false"
   ubi="false" eli="false" reflect="1.0" prefix="rh_" />
