Commit message: fixed xacro namespace declarations

File: sr_description/hand/xacro/finger/biotac/biotac.urdf.xacro (robot description, xacro)
@@ -1,9 +1,9 @@
 <robot xmlns:xacro="http://www.ros.org/wiki/xacro"
-xmlns:sensor="http://playerstage.sourceforge.net/gazebo/xmlschema/#sensor"
-xmlns:controller="http://playerstage.sourceforge.net/gazebo/xmlschema/#controller"
-xmlns:joint="http://playerstage.sourceforge.net/gazebo/xmlschema/#slider"
-xmlns:interface="http://playerstage.sourceforge.net/gazebo/xmlschema/#interface"
-xmlns:body="http://playerstage.sourceforge.net/gazebo/xmlschema/#body"
-xmlns:geom="http://playerstage.sourceforge.net/gazebo/xmlschema/#geom">
+        xmlns:sensor="http://playerstage.sourceforge.net/gazebo/xmlschema/#sensor"
+       xmlns:controller="http://playerstage.sourceforge.net/gazebo/xmlschema/#controller"
+       xmlns:joint="http://playerstage.sourceforge.net/gazebo/xmlschema/#slider"
+       xmlns:interface="http://playerstage.sourceforge.net/gazebo/xmlschema/#interface"
+       xmlns:body="http://playerstage.sourceforge.net/gazebo/xmlschema/#body"
+       xmlns:geom="http://playerstage.sourceforge.net/gazebo/xmlschema/#geom">
   <xacro:include filename="$(find sr_description)/hand/xacro/finger/middle/middle.transmission.xacro" />
   <!-- muscle is true for muscle hand or false for motor hand -->
@@ -17,5 +17,5 @@
       <inertial>
         <origin xyz="0 0 0.0125" rpy="0 0 0" />
-        <mass value="0.017" />
+          <mass value="0.017" />
         <inertia ixx="0.0000026" ixy="0.0" ixz="0.0"
         iyy="0.0000027" iyz="0.0" izz="0.00000087" />
@@ -143,10 +143,10 @@
       <origin xyz="0 0.0 0.008" rpy="0 0 0" />
     </joint>
-    <!-- extra link to imaginary sphere in fingertip for FK/IK calculations -->
+  <!-- extra link to imaginary sphere in fingertip for FK/IK calculations -->
     <!-- remove visual and collision once the correct position is found -->
     <link name="${prefix}${link_prefix}tip">
       <inertial>
-        <mass value="0.001" />
-        <origin xyz="0 0 0" rpy="0 0 0" />
+       <mass value="0.001" />
+       <origin xyz="0 0 0" rpy="0 0 0" />
         <inertia ixx="0.0" ixy="0.0" ixz="0.0" iyy="0.0" iyz="0.0"
         izz="0.0" />

File: sr_description/hand/xacro/thumb/thdistal.urdf.xacro (robot description, xacro)
@@ -1,13 +1,13 @@
 <robot xmlns:xacro="http://www.ros.org/wiki/xacro"
-xmlns:sensor="http://playerstage.sourceforge.net/gazebo/xmlschema/#sensor"
-xmlns:controller="http://playerstage.sourceforge.net/gazebo/xmlschema/#controller"
-xmlns:joint="http://playerstage.sourceforge.net/gazebo/xmlschema/#slider"
-xmlns:interface="http://playerstage.sourceforge.net/gazebo/xmlschema/#interface"
-xmlns:body="http://playerstage.sourceforge.net/gazebo/xmlschema/#body"
-xmlns:geom="http://playerstage.sourceforge.net/gazebo/xmlschema/#geom">
+       xmlns:sensor="http://playerstage.sourceforge.net/gazebo/xmlschema/#sensor"
+       xmlns:controller="http://playerstage.sourceforge.net/gazebo/xmlschema/#controller"
+       xmlns:joint="http://playerstage.sourceforge.net/gazebo/xmlschema/#slider"
+       xmlns:interface="http://playerstage.sourceforge.net/gazebo/xmlschema/#interface"
+       xmlns:body="http://playerstage.sourceforge.net/gazebo/xmlschema/#body"
+       xmlns:geom="http://playerstage.sourceforge.net/gazebo/xmlschema/#geom">
   <xacro:include filename="$(find sr_description)/hand/xacro/thumb/thdistal.gazebo.xacro" />
   <xacro:include filename="$(find sr_description)/hand/xacro/thumb/thdistal.transmission.xacro" />
   <!-- muscle is true for muscle hand or false for motor hand -->
-  <!-- bio is true for biotac finger or false for standard finger -->
+	<!-- bio is true for biotac finger or false for standard finger -->
   <!-- bt_sp is true for BT_SP finger or false for standard finger -->
   <!-- ubi is true for ubi finger or false for standard finger -->
@@ -17,8 +17,8 @@
   <xacro:macro name="thdistal"
   params="muscle bio bt_sp ubi eli prefix parent">
-    <xacro:if value="${bio}">
+		<xacro:if value="${bio}">
       <!--    BIOTAC -->
       <link name="${prefix}thdistal_J1_dummy">
-        <inertial>
+				<inertial>
           <origin xyz="0 0 0" rpy="0 0 0" />
           <mass value="0.001" />
@@ -26,75 +26,75 @@
           iyy="0.00000001" iyz="0.0" izz="0.00000001" />
         </inertial>
-      </link>
-      <joint name="${prefix}THJ1" type="revolute">
+			</link>
+			<joint name="${prefix}THJ1" type="revolute">
         <parent link="${parent}" />
         <child link="${prefix}thdistal_J1_dummy" />
-        <origin xyz="0 0 0.02" rpy="0 0 ${-M_PI/2}" />
-        <axis xyz="1 0 0" />
+				<origin xyz="0 0 0.02" rpy="0 0 ${-M_PI/2}" />
+				<axis xyz="1 0 0" />
         <limit lower="${20*M_PI/180}" upper="${20.1*M_PI/180}"
         effort="0.0" velocity="2.0" />
         <dynamics damping="0.5" />
-      </joint>
-      <gazebo reference="${prefix}THJ1">
-        <provideFeedback>1</provideFeedback>
-        <implicitSpringDamper>1</implicitSpringDamper>
-      </gazebo>
+			</joint>
+			<gazebo reference="${prefix}THJ1">
+				<provideFeedback>1</provideFeedback>
+				<implicitSpringDamper>1</implicitSpringDamper>
+			</gazebo>
       <link name="${prefix}thdistal">
-        <inertial>
+				<inertial>
           <origin xyz="-0.009 0.0 0.035" rpy="0 0 ${-M_PI/2}" />
           <!-- approximated only FIXME -->
-          <mass value="0.008" />
+					<mass value="0.008" />
           <inertia ixx="0.0000011" ixy="0.0" ixz="0.0"
           iyy="0.0000011" iyz="0.0" izz="0.0000005" />
-        </inertial>
-        <visual>
-          <origin xyz="0 0 0" rpy="0 0 0" />
+				</inertial>
+				<visual>
+					<origin xyz="0 0 0" rpy="0 0 0" />
           <geometry name="${prefix}th_distal_visual">
-            <!-- <mesh filename="package://sr_description/hand/model/biotacs/biotac.stl" scale="0.0254 0.0254 0.0254" /> -->
+						<!-- <mesh filename="package://sr_description/hand/model/biotacs/biotac.stl" scale="0.0254 0.0254 0.0254" /> -->
             <mesh filename="package://sr_description/hand/model/biotacs/biotac_decimated.dae"
             scale="0.0254 0.0254 0.0254" />
-          </geometry>
-          <material name="BiotacGreen" />
-        </visual>
-        <collision>
+					</geometry>
+					<material name="BiotacGreen" />
+				</visual>
+				<collision>
           <geometry name="${prefix}th_distal_collision_geom">
-            <!-- <box size="0.001 0.001 0.001" /> -->
-            <!-- <mesh filename="package://sr_description/hand/model/biotacs/biotac-v5.stl" scale="0.0254 0.0254 0.0254" /> -->
+						<!-- <box size="0.001 0.001 0.001" /> -->
+						<!-- <mesh filename="package://sr_description/hand/model/biotacs/biotac-v5.stl" scale="0.0254 0.0254 0.0254" /> -->
             <mesh filename="package://sr_description/hand/model/biotacs/biotac_decimated.dae"
             scale="0.0254 0.0254 0.0254" />
-          </geometry>
-        </collision>
-      </link>
-      <gazebo reference="${prefix}thdistal">
-        <sensor type="contact" name="${prefix}thdistal_contact">
-          <always_on>1</always_on>
-          <update_rate>1000.0</update_rate>
-          <contact>
+					</geometry>
+				</collision>
+			</link>
+			<gazebo reference="${prefix}thdistal">
+				<sensor type="contact" name="${prefix}thdistal_contact">
+					<always_on>1</always_on>
+					<update_rate>1000.0</update_rate>
+					<contact>
             <collision>${prefix}thdistal_geom</collision>
             <topic>${prefix}thdistal_collision</topic>
-          </contact>
+					</contact>
           <plugin name="${prefix}thdistal_gazebo_ros_bumper_controller"
           filename="libgazebo_ros_bumper.so">
-            <alwaysOn>true</alwaysOn>
+						<alwaysOn>true</alwaysOn>
             <frameName>${prefix}thdistal</frameName>
-            <updateRate>100.0</updateRate>
+						<updateRate>100.0</updateRate>
             <bumperTopicName>
             contacts/${prefix}th/distal</bumperTopicName>
-          </plugin>
-        </sensor>
-        <selfCollide>true</selfCollide>
-        <material>BiotacGreen</material>
-      </gazebo>
+					</plugin>
+				</sensor>
+				<selfCollide>true</selfCollide>
+				<material>BiotacGreen</material>
+			</gazebo>
       <joint name="${prefix}th_distal_joint" type="fixed">
         <parent link="${prefix}thmiddle" />
         <child link="${prefix}thdistal" />
-        <origin xyz="0 0.0 0.01" rpy="0 0 ${-M_PI/2}" />
-      </joint>
-      <!-- extra link to imaginary sphere in fingertip for FK/IK calculations -->
-      <!-- remove visual and collision once the correct position is found -->
-      <link name="${prefix}thtip">
-        <inertial>
-          <mass value="0.001" />
-          <origin xyz="0 0 0" rpy="0 0 0" />
+				<origin xyz="0 0.0 0.01" rpy="0 0 ${-M_PI/2}" />
+			</joint>
+		  <!-- extra link to imaginary sphere in fingertip for FK/IK calculations -->
+			<!-- remove visual and collision once the correct position is found -->
+			<link name="${prefix}thtip">
+				<inertial>
+				 <mass value="0.001" />
+				 <origin xyz="0 0 0" rpy="0 0 0" />
           <inertia ixx="0" ixy="0" ixz="0" iyy="0" iyz="0"
           izz="0" />
@@ -116,25 +116,25 @@
         <!-- approximated only FIXME -->
       </joint>
-    </xacro:if>
-    <xacro:unless value="${bio}">
-      <!-- common -->
-      <link name="${prefix}thdistal">
-        <inertial>
-          <mass value="0.016" />
+		</xacro:if>
+			<xacro:unless value="${bio}">
+				<!-- common -->
+				<link name="${prefix}thdistal">
+				<inertial>
+					<mass value="0.016" />
           <origin xyz="0 0 0.01375" rpy="0 0 0" />
           <inertia ixx="0.0000021" ixy="0.0" ixz="0.0"
           iyy="0.0000022" iyz="0.0" izz="0.000001" />
-        </inertial>
-        <visual>
-          <origin xyz="0 0 0" rpy="0 0 0" />
-          <geometry name="${prefix}thdistal_visual">
-            <xacro:if value="${eli}">
-              <!-- Ellispoid distal  -->
+				</inertial>
+				<visual>
+					<origin xyz="0 0 0" rpy="0 0 0" />
+					<geometry name="${prefix}thdistal_visual">
+						<xacro:if value="${eli}">
+							<!-- Ellispoid distal  -->
               <mesh filename="package://sr_description/hand/model/ellipsoids/thdistal_ellipsoid_visual.dae"
               scale="0.001 0.001 0.001" />
             </xacro:if>
-            <xacro:unless value="${eli}">
-              <xacro:if value="${ubi}">
-                <!-- Ubi distal -->
+						<xacro:unless value="${eli}">
+							<xacro:if value="${ubi}">
+								<!-- Ubi distal -->
                 <mesh filename="package://sr_description/hand/model/TH1_z.dae"
                       scale="0.001 0.001 0.001" />
@@ -146,5 +146,5 @@
 		</xacro:if>
 		<xacro:unless value="${bt_sp}">
-		  <!-- Standard distal  -->
+							<!-- Standard distal  -->
                   <mesh filename="package://sr_description/hand/model/TH1_z.dae"
 			scale="0.001 0.001 0.001" />
@@ -152,24 +152,24 @@
 	      </xacro:unless>
             </xacro:unless>
-          </geometry>
-          <material name="shadow_thmiddle_material">
+					</geometry>
+					<material name="shadow_thmiddle_material">
             <color rgba="0.2 0.2 0.2 1.0" />
-          </material>
-        </visual>
-        <collision>
+					</material>
+				</visual>
+				<collision>
           <origin xyz="0 0 0" rpy="0 0 0" />
-          <geometry name="${prefix}thmiddle_collision_geom">
-            <xacro:if value="${eli}">
-              <!-- Ellispoid distal  -->
+					<geometry name="${prefix}thmiddle_collision_geom">
+						<xacro:if value="${eli}">
+							<!-- Ellispoid distal  -->
               <mesh filename="package://sr_description/hand/model/ellipsoids/thdistal_ellipsoid.dae"
               scale="0.001 0.001 0.001" />
             </xacro:if>
-            <xacro:unless value="${eli}">
-              <xacro:if value="${ubi}">
-                <!-- Ubi distal -->
+						<xacro:unless value="${eli}">
+							<xacro:if value="${ubi}">
+								<!-- Ubi distal -->
                 <mesh filename="package://sr_description/hand/model/TH1_z.dae"
                 scale="0.001 0.001 0.001" />
               </xacro:if>
-              <xacro:unless value="${ubi}">
+							<xacro:unless value="${ubi}">
 		<xacro:if value="${bt_sp}">
 		  <!-- bt sp distal  -->
@@ -177,5 +177,5 @@
 		</xacro:if>
 		<xacro:unless value="${bt_sp}">
-                  <!-- Standard distal  -->
+								<!-- Standard distal  -->
                   <mesh filename="package://sr_description/hand/model/TH1_z.dae"
 			scale="0.001 0.001 0.001" />
@@ -184,35 +184,35 @@
             </xacro:unless>
             <!--      <box size="0.015 0.015 0.015" /> -->
-          </geometry>
-        </collision>
-      </link>
-      <joint name="${prefix}THJ1" type="revolute">
+					</geometry>
+				</collision>
+			</link>
+			<joint name="${prefix}THJ1" type="revolute">
         <parent link="${parent}" />
         <child link="${prefix}thdistal" />
-        <origin xyz="0 0 0.032" rpy="0 0 ${-M_PI/2}" />
-        <axis xyz="1 0 0" />
+				<origin xyz="0 0 0.032" rpy="0 0 ${-M_PI/2}" />
+				<axis xyz="1 0 0" />
         <limit lower="0" upper="${90.0*M_PI/180}" effort="1.0"
         velocity="4.0" />
         <dynamics damping="0.2" />
-      </joint>
-      <gazebo reference="${prefix}THJ1">
-        <provideFeedback>1</provideFeedback>
-        <implicitSpringDamper>1</implicitSpringDamper>
-      </gazebo>
-      <link name="${prefix}thtip">
-        <inertial>
-          <mass value="0.001" />
+			</joint>
+			<gazebo reference="${prefix}THJ1">
+				<provideFeedback>1</provideFeedback>
+				<implicitSpringDamper>1</implicitSpringDamper>
+			</gazebo>
+			<link name="${prefix}thtip">
+				<inertial>
+					<mass value="0.001" />
           <inertia ixx="0.0" ixy="0.0" ixz="0.0" iyy="0.0"
           iyz="0.0" izz="0.0" />
-        </inertial>
-      </link>
-      <joint name="${prefix}thtip" type="fixed">
+				</inertial>
+			</link>
+			<joint name="${prefix}thtip" type="fixed">
         <parent link="${prefix}thdistal" />
         <child link="${prefix}thtip" />
-        <origin xyz="0 0 0.0275" rpy="0 0 0" />
-      </joint>
-      <xacro:thdistal_gazebo prefix="${prefix}" />
+				<origin xyz="0 0 0.0275" rpy="0 0 0" />
+			</joint>
+			<xacro:thdistal_gazebo prefix="${prefix}" />
     </xacro:unless>
-    <!-- extensions -->
+		<!-- extensions -->
     <xacro:thdistal_transmission muscletrans="${muscle}"
     prefix="${prefix}" />
