Commit message: Added thumbtip model and markers for ubi distal, and changed distal xacro to use it

File: sr_description/hand/xacro/thumb/thdistal.urdf.xacro (robot description, xacro)
@@ -137,5 +137,5 @@
               <xacro:if value="${ubi}">
                 <!-- Ubi distal -->
-                <mesh filename="package://sr_description/hand/model/TH1_z.dae"
+                <mesh filename="package://sr_description/hand/model/ubi_tactiles/ubi_thtip_visual.dae"
                       scale="0.001 0.001 0.001" />
               </xacro:if>
@@ -168,5 +168,5 @@
               <xacro:if value="${ubi}">
                 <!-- Ubi distal -->
-                <mesh filename="package://sr_description/hand/model/TH1_z.dae"
+                <mesh filename="package://sr_description/hand/model/ubi_tactiles/ubi_thtip_collision.stl"
                 scale="0.001 0.001 0.001" />
               </xacro:if>

Commit message: Added thumbtip model and markers for ubi distal, and changed distal xacro to use it

File: sr_description/hand/xacro/thumb/thdistal.urdf.xacro (robot description, xacro)
@@ -137,5 +137,5 @@
 							<xacro:if value="${ubi}">
 								<!-- Ubi distal -->
-                <mesh filename="package://sr_description/hand/model/TH1_z.dae"
+                <mesh filename="package://sr_description/hand/model/ubi_tactiles/ubi_thtip_visual.dae"
                       scale="0.001 0.001 0.001" />
               </xacro:if>
@@ -168,5 +168,5 @@
 							<xacro:if value="${ubi}">
 								<!-- Ubi distal -->
-                <mesh filename="package://sr_description/hand/model/TH1_z.dae"
+                <mesh filename="package://sr_description/hand/model/ubi_tactiles/ubi_thtip_collision.stl"
                 scale="0.001 0.001 0.001" />
               </xacro:if>
