Commit message: reworked tactile marker description for UBI taxels
added arrow markers (taxel position+normals from yaml config)
prepared for thumb

File: sr_description/hand/xacro/full_hand.tactile.xacro (robot description, xacro)
@@ -1,24 +1,64 @@
-<robot xmlns:sensor="http://playerstage.sourceforge.net/gazebo/xmlschema/#sensor"
-       xmlns:controller="http://playerstage.sourceforge.net/gazebo/xmlschema/#controller"
-       xmlns:interface="http://playerstage.sourceforge.net/gazebo/xmlschema/#interface"
-       xmlns:xacro="http://www.ros.org/wiki/xacro">
-  <xacro:include filename="$(find sr_description)/hand/xacro/palm/palm.tactile.xacro" />
-  <xacro:include filename="$(find sr_description)/hand/xacro/finger/fingers.tactile.xacro" />
-  <property name="M_PI" value="3.1415926535897931" />
-  <!-- bio is true for biotac finger or false for standard finger -->
-  <!-- ubi is true for ubi finger or false for standard finger -->
-  <!-- eli is true for ellipsoid fingertip or false for standard finger -->
-  <!-- prefix can be anything but usually is "r_" or  "l_" for right and left hands distinction -->
-  <xacro:macro name="shadowhand_tactile" params="bio ubi eli reflect prefix">
+<robot xmlns:xacro="http://www.ros.org/wiki/xacro">
+  <!-- Create mesh and arrow markers for a single taxel.
+       Expected parameters:
+       meshes + normals = 0 | 1
+       topic: ROS topic
+       data: data field in ROS topic stream
+       link: link name
+       ns:   marker namespace in rviz
+       xs:   raw sensor range
+       mesh: mesh resource
+       mesh_scale: 3-dim vector for mesh scaling
+       normal_scale
+  -->
+  <xacro:macro name="xacro:tactile" params="topic data link ns xs
+                                            mesh mesh_scale arrow_scale
+                                            meshes normals">
+    <!-- extract channel number -->
+    <xacro:property name="channel" value="${data[:-1].rsplit('[',1)[1]}"/>
+    <xacro:if value="${meshes}">
+      <!-- mesh marker -->
+      <tactile topic="${topic}" data="${data}"
+               link="${link}" ns="meshes/${ns}" xs="${xs}">
+        <origin xyz="0 0 0" rpy="0 0 0"/>
+        <geometry>
+          <mesh filename="${mesh}" scale="${mesh_scale}" />
+        </geometry>
+      </tactile>
+    </xacro:if>
+    <xacro:if value="${normals}">
+      <!-- arrow marker -->
+      <tactile topic="${topic}" data="${data}" link="${link}" ns="normals/${ns}" xs="${xs}">
+        <origin xyz="${' '.join([str(v) for v in taxel_data['positions'][channel]])}"/>
+        <geometry>
+          <arrow dir="${' '.join([str(v) for v in taxel_data['normals'][channel]])}"
+                 scale="${arrow_scale}"/>
+        </geometry>
+      </tactile>
+    </xacro:if>
+  </xacro:macro>
+  <!-- Create <tactile> tags describing the taxels
+       tactile: sensor type
+       prefix:  hand prefix, usually rh_ or lh_
+       reflect: +1 / -1 to indicate right / left hand
+       meshes:  create tags for mesh markers?
+       normals: create tags for arrow markers?
+  -->
+  <xacro:macro name="shadowhand_tactile" params="tactile reflect:=1 prefix:='' meshes normals">
+    <xacro:include filename="$(find sr_description)/hand/xacro/palm/palm.tactile.${tactile}.xacro"/>
+    <xacro:include filename="$(find sr_description)/hand/xacro/finger/fingers.tactile.${tactile}.xacro"/>
+    <xacro:include filename="$(find sr_description)/hand/xacro/thumb/thumb.tactile.${tactile}.xacro"/>
     <!-- Palm -->
-    <xacro:palm_tactile reflect="${reflect}" prefix="${prefix}" />
+    <xacro:palm_tactile normals="0"/>
     <!-- First Finger -->
-    <xacro:finger_tactile lf="false" bio="${bio}" ubi="${ubi}" eli="${eli}" reflect="${reflect}" prefix="${prefix}" link_prefix="ff"  finger_number="0"/>
+    <xacro:finger_tactile finger="ff"/>
     <!-- Middle Finger -->
-    <xacro:finger_tactile lf="false" bio="${bio}" ubi="${ubi}" eli="${eli}" reflect="${reflect}" prefix="${prefix}" link_prefix="mf"  finger_number="1"/>
+    <xacro:finger_tactile finger="mf"/>
     <!-- Ring Finger -->
-    <xacro:finger_tactile lf="false" bio="${bio}" ubi="${ubi}" eli="${eli}" reflect="${reflect}" prefix="${prefix}" link_prefix="rf"  finger_number="2"/>
+    <xacro:finger_tactile finger="rf"/>
     <!-- Little Finger  -->
-    <xacro:finger_tactile lf="true" bio="${bio}" ubi="${ubi}" eli="${eli}" reflect="${reflect}" prefix="${prefix}" link_prefix="lf"  finger_number="3"/>
+    <xacro:finger_tactile finger="lf"/>
+    <!-- Thumb  -->
+    <xacro:thumb_tactile/>
   </xacro:macro>
 </robot>

Commit message: Migrate to new tactile representation in sensors, use orientations instead of normals

File: sr_description/hand/xacro/full_hand.tactile.xacro (robot description, xacro)
@@ -4,9 +4,7 @@
        prefix:  hand prefix, usually rh_ or lh_
        reflect: +1 / -1 to indicate right / left hand
-       meshes:  create tags for mesh markers?
-       normals: create tags for arrow markers?
   -->
   <xacro:macro name="shadowhand_tactile"
-               params="tactile:=^ reflect:=^|1 prefix:=^|'' meshes:=^ normals:=^">
+               params="tactile:=^ reflect:=^|1 prefix:=^|''">
     <xacro:if value="${tactile in ['ubi']}">
       <!-- load macros specific to sensor type -->

File: sr_description/hand/xacro/tactile.ubi.xacro (robot description, xacro)
@@ -8,12 +8,7 @@
     <xacro:property name="mesh_dir" value="package://sr_description/hand/model/ubi_tactiles" scope="parent"/>
     <xacro:property name="mesh_scale" value="0.00101 0.00101 0.00101" scope="parent"/>
-    <xacro:property name="origin" scope="parent"><origin xyz="0 0 0" rpy="0 0 0"/></xacro:property>
-    <!-- arrow parameters -->
-    <xacro:property name="arrow_scale" value="0.01 0.0005 0.001" scope="parent"/>
+    <!-- <xacro:property name="origin" scope="parent"><origin xyz="0 0 0" rpy="0 0 0"/></xacro:property>-->
     <xacro:if value="${link == ''}">
       <xacro:property name="link" value="${prefix}${finger}${_link}" scope="parent"/>
-    </xacro:if>
-    <xacro:if value="${ns == ''}">
-      <xacro:property name="ns" value="${prefix}${finger}" scope="parent"/>
     </xacro:if>
   </xacro:macro>
@@ -22,59 +17,67 @@
        accept the following arguments:
        taxel_data: positions + normals
-       topic:      ROS topic
-       data:       data field in topic
+       tactile_name: unique name of the sensor
        link:       link name
-       ns:         marker group namespace (for rviz enabling/disabling)
-       xs:         sensor range
        prefix:  hand prefix, usually rh_ or lh_
        finger:  finger name (ff, mf, rf, lf, th)
        reflect: +1 / -1 to indicate right / left hand
-       meshes:  create tags for mesh markers?
-       normals: create tags for arrow markers?
   -->
   <xacro:macro name="proximal_tactile"
-               params="taxel_data topic:=tactile_mid_prox link:='' ns:='' xs:=^
-                       prefix:=^|'' reflect:=^|1 finger:=^
-                       meshes:=^|1 normals:=^|1">
+               params="taxel_data tactile_name:=proximal link:=''
+                       prefix:=^|'' reflect:=^|1 finger:=^">
     <xacro:tactile_default_params _link="proximal"/>
-    <xacro:property name="data" value="sensors[${finger_no[finger]}]/proximal"/>
-    <xacro:taxel data="${data}[0]"  mesh="${mesh_dir}/tax_prox_r.stl"/>
-    <xacro:taxel data="${data}[1]" mesh="${mesh_dir}/tax_prox_m.stl"/>
-    <xacro:taxel data="${data}[2]" mesh="${mesh_dir}/tax_prox_l.stl"/>
+    <xacro:property name="name" value="${prefix}${finger}${tactile_name}"/>
+    <sensor name="${name}" update_rate="100" >
+      <parent link="${link}" />
+      <origin xyz="0 0 0" rpy="0 0 0"/>
+      <tactile>
+        <xacro:taxel_macro idx="0" mesh="${mesh_dir}/tax_prox_r.stl"/>
+        <xacro:taxel_macro idx="1" mesh="${mesh_dir}/tax_prox_m.stl"/>
+        <xacro:taxel_macro idx="2" mesh="${mesh_dir}/tax_prox_l.stl"/>
+      </tactile>
+    </sensor>
   </xacro:macro>
   <xacro:macro name="middle_tactile"
-               params="taxel_data topic:=tactile_mid_prox link:='' ns:='' xs:=^
-                       prefix:=^|'' reflect:=^|1 finger:=^
-                       meshes:=^|1 normals:=^|1">
+               params="taxel_data tactile_name:=middle link:=''
+                       prefix:=^|'' reflect:=^|1 finger:=^">
     <xacro:tactile_default_params _link="middle"/>
-    <xacro:property name="data" value="sensors[${finger_no[finger]}]/middle"/>
-    <xacro:taxel data="${data}[0]" mesh="${mesh_dir}/tax_mid_l.stl"/>
-    <xacro:taxel data="${data}[1]" mesh="${mesh_dir}/tax_mid_r.stl"/>
+    <xacro:property name="name" value="${prefix}${finger}${tactile_name}"/>
+    <sensor name="${name}" update_rate="100" >
+      <parent link="${link}" />
+      <origin xyz="0 0 0" rpy="0 0 0"/>
+      <tactile>
+        <xacro:taxel_macro idx="0" mesh="${mesh_dir}/tax_mid_l.stl"/>
+        <xacro:taxel_macro idx="1" mesh="${mesh_dir}/tax_mid_r.stl"/>
+      </tactile>
+    </sensor>
   </xacro:macro>
   <xacro:macro name="distal_tactile"
-               params="taxel_data topic:=tactile link:='' ns:='' xs:=^
-                       prefix:=^|'' reflect:=^|1 finger:=^
-                       meshes:=^|1 normals:=^|1">
+               params="taxel_data tactile_name:=distal link:=''
+                       prefix:=^|'' reflect:=^|1 finger:=^">
     <xacro:tactile_default_params _link="distal"/>
+    <xacro:property name="name" value="${prefix}${finger}${tactile_name}"/>
     <xacro:property name="tipname" value="${'thtip' if finger=='th' else 'tip'}"/>
-    <xacro:property name="data" value="tactiles[${finger_no[finger]}]/distal"/>
-    <xacro:taxel data="${data}[0]" mesh="${mesh_dir}/tax_${tipname}_0.stl"/>
-    <xacro:taxel data="${data}[1]" mesh="${mesh_dir}/tax_${tipname}_1.stl"/>
-    <xacro:taxel data="${data}[2]" mesh="${mesh_dir}/tax_${tipname}_2.stl"/>
-    <xacro:taxel data="${data}[3]" mesh="${mesh_dir}/tax_${tipname}_3.stl"/>
-    <xacro:taxel data="${data}[4]" mesh="${mesh_dir}/tax_${tipname}_4.stl"/>
-    <xacro:taxel data="${data}[5]" mesh="${mesh_dir}/tax_${tipname}_5.stl"/>
-    <xacro:taxel data="${data}[6]" mesh="${mesh_dir}/tax_${tipname}_6.stl"/>
-    <xacro:taxel data="${data}[7]" mesh="${mesh_dir}/tax_${tipname}_7.stl"/>
-    <xacro:taxel data="${data}[8]" mesh="${mesh_dir}/tax_${tipname}_8.stl"/>
-    <xacro:taxel data="${data}[9]" mesh="${mesh_dir}/tax_${tipname}_9.stl"/>
-    <xacro:taxel data="${data}[10]" mesh="${mesh_dir}/tax_${tipname}_10.stl"/>
-    <xacro:taxel data="${data}[11]" mesh="${mesh_dir}/tax_${tipname}_11.stl"/>
+    <sensor name="${name}" update_rate="100" >
+      <parent link="${link}" />
+      <origin xyz="0 0 0" rpy="0 0 0"/>
+      <tactile>
+        <xacro:taxel_macro idx="0" mesh="${mesh_dir}/tax_${tipname}_0.stl"/>
+        <xacro:taxel_macro idx="1" mesh="${mesh_dir}/tax_${tipname}_1.stl"/>
+        <xacro:taxel_macro idx="2" mesh="${mesh_dir}/tax_${tipname}_2.stl"/>
+        <xacro:taxel_macro idx="3" mesh="${mesh_dir}/tax_${tipname}_3.stl"/>
+        <xacro:taxel_macro idx="4" mesh="${mesh_dir}/tax_${tipname}_4.stl"/>
+        <xacro:taxel_macro idx="5" mesh="${mesh_dir}/tax_${tipname}_5.stl"/>
+        <xacro:taxel_macro idx="6" mesh="${mesh_dir}/tax_${tipname}_6.stl"/>
+        <xacro:taxel_macro idx="7" mesh="${mesh_dir}/tax_${tipname}_7.stl"/>
+        <xacro:taxel_macro idx="8" mesh="${mesh_dir}/tax_${tipname}_8.stl"/>
+        <xacro:taxel_macro idx="9" mesh="${mesh_dir}/tax_${tipname}_9.stl"/>
+        <xacro:taxel_macro idx="10" mesh="${mesh_dir}/tax_${tipname}_10.stl"/>
+        <xacro:taxel_macro idx="11" mesh="${mesh_dir}/tax_${tipname}_11.stl"/>
+      </tactile>
+    </sensor>
   </xacro:macro>
   <xacro:macro name="finger_tactile"
-               params="prefix:=^|'' reflect:=^|1 finger
-                       meshes:=^|1 normals:=^|1">
+               params="prefix:=^|'' reflect:=^|1 finger">
     <xacro:property name="taxel_dir" value="$(find sr_description)/hand/xacro/finger"/>
-    <xacro:property name="xs" value="0 2047"/>
     <!-- Proximal -->
     <xacro:proximal_tactile taxel_data="${load_yaml(taxel_dir + '/proximal/proximal.taxels.ubi.yaml')}"/>
@@ -82,20 +85,16 @@
     <xacro:middle_tactile taxel_data="${load_yaml(taxel_dir + '/middle/middle.taxels.ubi.yaml')}"/>
     <!-- Distal -->
-    <xacro:property name="xs" value="1023 0"/>
     <xacro:distal_tactile taxel_data="${load_yaml(taxel_dir + '/distal/distal.taxels.ubi.yaml')}"/>
   </xacro:macro>
   <xacro:macro name="thumb_tactile"
-               params="prefix:=^|'' reflect:=^|1 meshes:=^|1 normals:=^|1">
+               params="prefix:=^|'' reflect:=^|1">
     <xacro:property name="taxel_dir" value="$(find sr_description)/hand/xacro/thumb"/>
     <!-- Distal  -->
-    <xacro:property name="xs" value="1023 0"/>
     <xacro:distal_tactile finger="th" taxel_data="${load_yaml(taxel_dir + '/thdistal.taxels.ubi.yaml')}"/>
   </xacro:macro>
   <xacro:macro name="palm_tactile"
-               params="prefix:=^|'' reflect:=^|1 meshes:=^|1 normals:=^|1 ns:=''">
+               params="prefix:=^|'' reflect:=^|1">
     <xacro:property name="taxel_dir" value="$(find sr_description)/hand/xacro/palm"/>
-    <xacro:property name="xs" value="0 2047"/>
     <xacro:property name="taxel_data" value="${load_yaml(taxel_dir + '/metacarpal.taxels.ubi.yaml')}"/>
-    <xacro:property name="topic" value="palm_extras"/>
     <xacro:property name="link" value="${prefix}lfmetacarpal"/>
     <!-- default finger and data properties to allow calling tactile_default_params -->
@@ -105,20 +104,31 @@
     <xacro:property name="mesh_scale" value="${reflect*0.00101} 0.00101 0.00101"/>
     <!-- taxels attached to lfmetacarpal -->
-    <xacro:taxel data="data[6]" mesh="${mesh_dir}/tax_metac_upper.stl"/>
-    <xacro:taxel data="data[7]" mesh="${mesh_dir}/tax_metac_lower.stl"/>
-    <xacro:taxel data="data[8]" mesh="${mesh_dir}/tax_metac_side.stl"/>
+    <sensor name="${prefix}lfmetacarpal" update_rate="100" >
+      <parent link="${link}" />
+      <origin xyz="0 0 0" rpy="0 0 0"/>
+      <tactile>
+        <xacro:taxel_macro idx="0" mesh="${mesh_dir}/tax_metac_upper.stl"/>
+        <xacro:taxel_macro idx="1" mesh="${mesh_dir}/tax_metac_lower.stl"/>
+        <xacro:taxel_macro idx="2" mesh="${mesh_dir}/tax_metac_side.stl"/>
+      </tactile>
+    </sensor>
     <!-- taxels attached to palm -->
+    <xacro:property name="taxel_data" value="${load_yaml(taxel_dir + '/palm.taxels.ubi.yaml')}"/>
     <xacro:property name="link" value="${prefix}palm"/>
-    <xacro:taxel data="data[9]" mesh="${mesh_dir}/tax_palm_side.stl"/>
-    <xacro:property name="taxel_data" value="${load_yaml(taxel_dir + '/palm.taxels.ubi.yaml')}"/>
-    <xacro:property name="topic" value="tactile_aux_spi"/>
-    <xacro:taxel data="sensors[0]" mesh="${mesh_dir}/tax_palm_up_r.stl"/>
-    <xacro:taxel data="sensors[1]" mesh="${mesh_dir}/tax_palm_up_mid.stl"/>
-    <xacro:taxel data="sensors[2]" mesh="${mesh_dir}/tax_palm_up_l.stl"/>
-    <xacro:taxel data="sensors[3]" mesh="${mesh_dir}/tax_palm_center_r.stl"/>
-    <xacro:taxel data="sensors[4]" mesh="${mesh_dir}/tax_palm_center_l.stl"/>
-    <xacro:taxel data="sensors[5]" mesh="${mesh_dir}/tax_palm_center_mid.stl"/>
-    <xacro:taxel data="sensors[6]" mesh="${mesh_dir}/tax_palm_down_r.stl"/>
-    <xacro:taxel data="sensors[7]" mesh="${mesh_dir}/tax_palm_down_l.stl"/>
+    <sensor name="${prefix}palm" update_rate="100" >
+      <parent link="${link}" />
+      <origin xyz="0 0 0" rpy="0 0 0"/>
+      <tactile>
+        <xacro:taxel_macro idx="0" mesh="${mesh_dir}/tax_palm_up_r.stl"/>
+        <xacro:taxel_macro idx="1" mesh="${mesh_dir}/tax_palm_up_mid.stl"/>
+        <xacro:taxel_macro idx="2" mesh="${mesh_dir}/tax_palm_up_l.stl"/>
+        <xacro:taxel_macro idx="3" mesh="${mesh_dir}/tax_palm_center_r.stl"/>
+        <xacro:taxel_macro idx="4" mesh="${mesh_dir}/tax_palm_center_l.stl"/>
+        <xacro:taxel_macro idx="5" mesh="${mesh_dir}/tax_palm_center_mid.stl"/>
+        <xacro:taxel_macro idx="6" mesh="${mesh_dir}/tax_palm_down_r.stl"/>
+        <xacro:taxel_macro idx="7" mesh="${mesh_dir}/tax_palm_down_l.stl"/>
+        <xacro:taxel_macro idx="8" mesh="${mesh_dir}/tax_palm_side.stl"/>
+      </tactile>
+    </sensor>
   </xacro:macro>
 </robot>

File: sr_description/hand/xacro/taxel.xacro (robot description, xacro)
@@ -2,42 +2,19 @@
   <!-- Create mesh and arrow markers for a single taxel.
        Expected parameters:
-       topic: ROS topic
-       data: data field in ROS topic stream
-       link: link name
-       ns:   marker namespace in rviz
-       xs:   raw sensor range
-       taxel_data: dict of taxel positions and normals
+       idx: the index in the channelfloat32 values
+       taxel_data: dict of taxel positions and orientations
        mesh: mesh resource
        mesh_scale: 3-dim vector for mesh scaling
-       arrow_scale: 4-dim scaling vector:
-                    len scaling, shaft thickness, head thickness, head len
-       meshes + normals = 0 | 1
   -->
-  <xacro:macro name="xacro:taxel"
-               params="topic:=^ data link:=^ ns:=^ xs:=^ taxel_data:=^
-                       mesh:=^ mesh_scale:=^ arrow_scale:=^
-                       meshes:=^ normals:=^">
-    <!-- extract channel number from data -->
-    <xacro:property name="channel" value="${data[:-1].rsplit('[',1)[1]}"/>
-    <xacro:if value="${meshes}">
-      <!-- mesh marker -->
-      <tactile topic="${topic}" data="${data}"
-               link="${link}" ns="meshes/${ns}" xs="${xs}">
-        <origin xyz="0 0 0" rpy="0 0 0"/>
-        <geometry>
-          <mesh filename="${mesh}" scale="${mesh_scale}" />
-        </geometry>
-      </tactile>
-    </xacro:if>
-    <xacro:if value="${normals}">
-      <!-- arrow marker -->
-      <tactile topic="${topic}" data="${data}" link="${link}" ns="normals/${ns}" xs="${xs}">
-        <origin xyz="${' '.join([str(v) for v in taxel_data['positions'][channel]])}"/>
-        <geometry>
-          <arrow dir="${' '.join([str(v) for v in taxel_data['normals'][channel]])}"
-                 scale="${arrow_scale}"/>
-        </geometry>
-      </tactile>
-    </xacro:if>
+  <xacro:macro name="xacro:taxel_macro"
+               params="idx taxel_data:=^
+                       mesh:=^ mesh_scale:=^">
+    <taxel idx="${idx}">
+      <origin xyz="${' '.join([str(v) for v in taxel_data['positions'][idx]])}"
+              rpy="${' '.join([str(v) for v in taxel_data['orientations'][idx]])}" />
+      <geometry>
+        <mesh filename="${mesh}" scale="${mesh_scale}" />
+      </geometry>
+    </taxel>
   </xacro:macro>
 </taxel>
