Commit message: Adapted taxel macro to match new attributes

File: sr_description/hand/xacro/taxel.xacro (robot description, xacro)
@@ -10,7 +10,7 @@
                params="idx taxel_data:=^
                        mesh:=^ mesh_scale:=^">
-    <taxel idx="${idx}">
-      <origin xyz="${' '.join([str(v) for v in taxel_data['positions'][idx]])}"
-              rpy="${' '.join([str(v) for v in taxel_data['orientations'][idx]])}" />
+    <taxel idx="${idx}"
+           xyz="${' '.join([str(v) for v in taxel_data['positions'][idx]])}"
+           rpy="${' '.join([str(v) for v in taxel_data['orientations'][idx]])}">
       <geometry>
         <mesh filename="${mesh}" scale="${mesh_scale}" />

Commit message: name of the macro should not contain xacro

File: sr_description/hand/xacro/taxel.xacro (robot description, xacro)
@@ -7,5 +7,5 @@
        mesh_scale: 3-dim vector for mesh scaling
   -->
-  <xacro:macro name="xacro:taxel_macro"
+  <xacro:macro name="taxel_macro"
                params="idx taxel_data:=^
                        mesh:=^ mesh_scale:=^">
