Commit message: Support sensor selection, to permit deactivating gazebo sensors and simplified xacro docs using latest xacro features

File: sr_description/hand/xacro/ff_biotac_hand.urdf.xacro (robot description, xacro)
@@ -11,58 +11,49 @@
   <!-- muscletrans is true for muscle transmission to be used, false to use motor transmission -->
   <!-- muscle is true for muscle hand or false for motor hand -->
-  <!-- bio is true for biotac finger or false for standard finger -->
-  <!-- bt_sp is true for BT_SP finger or false for standard finger -->
-  <!-- ubi is true for ubi finger or false for standard finger -->
-  <!-- eli is true for ellipsoid fingertip or false for standard finger -->
+  <!-- bio (deprecated) is true for biotac finger or false for standard finger -->
+  <!-- bt_sp (deprecated) is true for BT_SP finger or false for standard finger -->
+  <!-- ubi (deprecated) is true for ubi finger or false for standard finger -->
+  <!-- eli (deprecated) is true for ellipsoid fingertip or false for standard finger -->
+  <!-- tip_sensor describes the sensor none, bio, bt_sp, ubi, eli -->
+  <!-- mid_sensor describes the sensor none, bio, ubi -->
+  <!-- prox_sensor describes the sensor none, bumper, ubi -->
+  <!-- palm_sensor describes the sensor none, bumper, ubi -->
   <!-- reflect is either 1 (for right hand) or -1 (for left hand) -->
   <!-- prefix can be anything but usually is "r_" or  "l_" for right and left hands distinction -->
   <xacro:macro name="shadowhand"
-  params="muscletrans muscle bio bt_sp ubi eli reflect prefix">
+  params="muscletrans muscle bio:=False bt_sp:=False ubi:=False eli:=False tip_sensor:=bumper prox_sensor:=bumper mid_sensor:=bumper palm_sensor:=bumper reflect prefix">
+    <xacro:include filename="$(find sr_description)/hand/xacro/backward_compat.urdf.xacro" />
     <!-- Forearm -->
-    <xacro:forearm muscle="${muscle}" prefix="${prefix}" />
+    <xacro:forearm />
     <!-- Wrist -->
     <xacro:if value="${muscle}">
-      <xacro:wrist muscletrans="${muscletrans}" prefix="${prefix}"
-      reflect="${reflect}" parent="${prefix}forearm">
+      <xacro:wrist parent="${prefix}forearm">
         <origin xyz="0 0 0.4096" rpy="0 0 0" />
       </xacro:wrist>
     </xacro:if>
     <xacro:unless value="${muscle}">
-      <xacro:wrist muscletrans="false" prefix="${prefix}"
-      reflect="${reflect}" parent="${prefix}forearm">
+      <xacro:wrist muscletrans="false" parent="${prefix}forearm">
         <origin xyz="0 -0.010 0.213" rpy="0 0 0" />
       </xacro:wrist>
     </xacro:unless>
     <!-- Palm -->
-    <xacro:palm muscletrans="${muscletrans}" prefix="${prefix}"
-    reflect="${reflect}" parent="${prefix}wrist" />
+    <xacro:palm parent="${prefix}wrist" />
     <!-- First Finger Biotac -->
-    <xacro:finger muscletrans="${muscletrans}" lf="false"
-    bio="true" bt_sp="false" ubi="false" eli="false" prefix="${prefix}"
-    reflect="${reflect}" link_prefix="ff" joint_prefix="FF"
-    parent="${prefix}palm">
+    <xacro:finger tip_sensor="bio" link_prefix="ff" joint_prefix="FF" parent="${prefix}palm">
       <origin xyz="${reflect*0.033} 0 0.095" rpy="0 0 0" />
       <axis xyz="0 ${-1*reflect} 0" />
     </xacro:finger>
     <!-- Middle Finger -->
-    <xacro:finger muscletrans="${muscletrans}" lf="false"
-    bio="${bio}" bt_sp="false" ubi="${ubi}" eli="${eli}" prefix="${prefix}"
-    reflect="${reflect}" link_prefix="mf" joint_prefix="MF"
-    parent="${prefix}palm">
+    <xacro:finger link_prefix="mf" joint_prefix="MF" parent="${prefix}palm">
       <origin xyz="${reflect*0.011} 0 0.099" rpy="0 0 0" />
       <axis xyz="0 ${-1*reflect} 0" />
     </xacro:finger>
     <!-- Ring Finger -->
-    <xacro:finger muscletrans="${muscletrans}" lf="false"
-    bio="${bio}" bt_sp="${bt_sp}" ubi="${ubi}" eli="${eli}" prefix="${prefix}"
-    reflect="${reflect}" link_prefix="rf" joint_prefix="RF"
-    parent="${prefix}palm">
+    <xacro:finger link_prefix="rf" joint_prefix="RF" parent="${prefix}palm">
       <origin xyz="${reflect*-0.011} 0 0.095" rpy="0 0 0" />
       <axis xyz="0 ${reflect} 0" />
     </xacro:finger>
     <!-- Little Finger  -->
-    <xacro:finger muscletrans="${muscletrans}" lf="true"
-    bio="${bio}" bt_sp="${bt_sp}" ubi="${ubi}" eli="${eli}" prefix="${prefix}"
-    reflect="${reflect}" link_prefix="lf" joint_prefix="LF"
+    <xacro:finger link_prefix="lf" joint_prefix="LF"
     parent="${prefix}palm">
       <origin xyz="0 0 0.06579" rpy="0 0 0" />
@@ -70,8 +61,5 @@
     </xacro:finger>
     <!-- Thumb Biotac -->
-    <xacro:thumb muscletrans="${muscletrans}" bio="${bio}" bt_sp="${bt_sp}"
-    ubi="${ubi}" eli="${eli}" prefix="${prefix}"
-    reflect="${reflect}" is_lite="0" parent="${prefix}palm">
-    </xacro:thumb>
+    <xacro:thumb is_lite="0" parent="${prefix}palm" />
   </xacro:macro>
 </robot>

File: sr_description/hand/xacro/finger/biotac/biotac.urdf.xacro (robot description, xacro)
@@ -13,5 +13,5 @@
   <!-- parent is the parent link for the joint -->
   <xacro:macro name="biotac_middle"
-  params="muscle prefix link_prefix joint_prefix parent">
+  params="muscle:=^ prefix:=^ link_prefix:=^ joint_prefix:=^ tip_sensor:=^|bumper mid_sensor:=^|standard parent">
     <link name="${prefix}${link_prefix}middle">
       <inertial>
@@ -37,4 +37,5 @@
     </link>
     <gazebo reference="${prefix}${link_prefix}middle">
+      <xacro:unless value="${'none' in mid_sensor}" >
       <sensor type="contact"
       name="${prefix}${link_prefix}middle_contact">
@@ -54,4 +55,5 @@
         </plugin>
       </sensor>
+      </xacro:unless>
       <material>Gazebo/FlatBlack</material>
     </gazebo>
@@ -90,7 +92,5 @@
       <implicitSpringDamper>1</implicitSpringDamper>
     </gazebo>
-    <xacro:middle_transmission muscletrans="${muscle}"
-    prefix="${prefix}" joint_prefix="${joint_prefix}"
-    link_prefix="${link_prefix}" />
+    <xacro:middle_transmission muscletrans="${muscle}" />
     <link name="${prefix}${link_prefix}distal">
       <inertial>
@@ -118,4 +118,5 @@
     </link>
     <gazebo reference="${prefix}${link_prefix}distal">
+      <xacro:unless value="${'none' in tip_sensor}" >
       <sensor type="contact"
       name="${prefix}${link_prefix}distal_contact">
@@ -135,4 +136,5 @@
         </plugin>
       </sensor>
+      </xacro:unless>
       <selfCollide>true</selfCollide>
     </gazebo>

File: sr_description/hand/xacro/finger/distal/distal.gazebo.xacro (robot description, xacro)
@@ -1,23 +1,43 @@
 <?xml version="1.0"?>
 <robot xmlns:xacro="http://www.ros.org/wiki/xacro">
-  <xacro:macro name="distal_gazebo" params="prefix link_prefix ns:=^|''">
-  <!-- prefix can be anything but usually is "rh_" or  "lh_" for right and left hands distinction -->
-  <gazebo reference="${prefix}${link_prefix}distal">
-      <sensor type="contact" name="${prefix}${link_prefix}distal_sensor">
-        <always_on>1</always_on>
-        <update_rate>1000.0</update_rate>
-        <contact>
-          <collision>${prefix}${link_prefix}distal_collision</collision>
-          <topic>${prefix}${link_prefix}distal_collision</topic>
-        </contact>
-        <plugin name="${prefix}${link_prefix}distal_gazebo_ros_tactile_controller" filename="libgazebo_ros_tactile.so">
-          <alwaysOn>true</alwaysOn>
-          <robotNamespace>${ns}</robotNamespace>
-          <frameName>${prefix}${link_prefix}distal</frameName>
-          <updateRate>100.0</updateRate>
-          <bumperTopicName>contacts/${prefix}${link_prefix}/distal</bumperTopicName>
-          <tactileTopicName>tactile_states/${prefix}${link_prefix}/distal</tactileTopicName>
-        </plugin>
-      </sensor>
+  <xacro:macro name="distal_gazebo" params="prefix:=^ link_prefix:=^ tip_sensor:=^|standard ns:=^|''">
+    <!-- prefix can be anything but usually is "rh_" or  "lh_" for right and left hands distinction -->
+    <gazebo reference="${prefix}${link_prefix}distal">
+      <xacro:unless value="${'none' in tip_sensor}" >
+        <xacro:if value="${'bumper' in tip_sensor}" >
+        <sensor type="contact" name="${prefix}${link_prefix}distal_contact">
+          <always_on>1</always_on>
+          <update_rate>1000.0</update_rate>
+          <contact>
+            <collision>${prefix}${link_prefix}distal_collision</collision>
+            <topic>${prefix}${link_prefix}distal_collision</topic>
+          </contact>
+          <plugin name="${prefix}${link_prefix}distal_gazebo_ros_bumper_controller" filename="libgazebo_ros_bumper.so">
+            <alwaysOn>true</alwaysOn>
+            <frameName>${prefix}${link_prefix}distal</frameName>
+            <updateRate>100.0</updateRate>
+            <bumperTopicName>contacts/${prefix}${link_prefix}/distal</bumperTopicName>
+          </plugin>
+        </sensor>
+        </xacro:if>
+        <xacro:if value="${'ubi' in tip_sensor}" >
+        <sensor type="contact" name="${prefix}${link_prefix}distal_sensor">
+          <always_on>1</always_on>
+          <update_rate>1000.0</update_rate>
+          <contact>
+            <collision>${prefix}${link_prefix}distal_collision</collision>
+            <topic>${prefix}${link_prefix}distal_collision</topic>
+          </contact>
+          <plugin name="${prefix}${link_prefix}distal_gazebo_ros_tactile_controller" filename="libgazebo_ros_tactile.so">
+            <alwaysOn>true</alwaysOn>
+            <robotNamespace>${ns}</robotNamespace>
+            <frameName>${prefix}${link_prefix}distal</frameName>
+            <updateRate>100.0</updateRate>
+            <bumperTopicName>contacts/${prefix}${link_prefix}/distal</bumperTopicName>
+            <tactileTopicName>tactile_states/${prefix}${link_prefix}/distal</tactileTopicName>
+          </plugin>
+        </sensor>
+        </xacro:if>
+      </xacro:unless>
       <mu1 value="500.0" />
       <mu2 value="500.0" />

File: sr_description/hand/xacro/finger/distal/distal.transmission.xacro (robot description, xacro)
@@ -8,5 +8,5 @@
   <!-- link_prefix prepends fingername to the link names -->
   <!-- joint_prefix prepends fingername to the joint names -->
-  <xacro:macro name="distal_transmission" params="muscletrans prefix joint_prefix link_prefix" >
+  <xacro:macro name="distal_transmission" params="muscletrans prefix:=^ joint_prefix:=^ link_prefix:=^" >
    <!-- muscle hand -->
     <xacro:if value="${muscletrans}">

File: sr_description/hand/xacro/finger/distal/distal.urdf.xacro (robot description, xacro)
@@ -9,8 +9,5 @@
   <xacro:include filename="$(find sr_description)/hand/xacro/finger/distal/distal.transmission.xacro" />
   <!-- muscle is true for muscle hand or false for motor hand -->
-  <!-- bio is true for biotac finger or false for standard finger -->
-  <!-- bt_sp is true for BT_SP finger or false for standard finger -->
-  <!-- ubi is true for ubi finger or false for standard finger -->
-  <!-- eli is true for ellipsoid fingertip or false for standard finger -->
+  <!-- tip_sensor describes the sensor none, bio, bt_sp, ubi, eli -->
   <!-- prefix can be anything but usually is "r_" or  "l_" for right and left hands distinction -->
   <!-- link_prefix prepends fingername to the link names -->
@@ -18,5 +15,5 @@
   <!-- parent is the parent link for the joint -->
   <xacro:macro name="distal"
-  params="muscle bio bt_sp ubi eli prefix link_prefix joint_prefix parent">
+  params="muscle:=^ prefix:=^ link_prefix:=^ joint_prefix:=^ tip_sensor:=^|standard parent">
     <link name="${prefix}${link_prefix}distal">
       <inertial>
@@ -29,34 +26,25 @@
         <origin xyz="0 0 0" rpy="0 0 0" />
         <geometry name="${prefix}${link_prefix}distal_visual">
-          <xacro:if value="${ubi}">
-            <!-- Ubi distal -->
-            <mesh filename="package://sr_description/hand/model/ubi_tactiles/ubi_tip_visual.dae"
-		  scale="0.001 0.001 0.001" />
-          </xacro:if>
-          <xacro:unless value="${ubi}">
-            <xacro:if value="${eli}">
+          <xacro:unless value="${tip_sensor in ['ubi','bt_sp','eli']}">
+            <!-- Standard distal  -->
+            <mesh filename="package://sr_description/hand/model/F1.dae"
+                  scale="0.001 0.001 0.001" />
+          </xacro:unless>
+          <xacro:if value="${tip_sensor in ['ubi','bt_sp','eli']}">
+            <xacro:if value="${'ubi' in tip_sensor}">
+              <!-- Ubi distal -->
+              <mesh filename="package://sr_description/hand/model/ubi_tactiles/ubi_tip_visual.dae"
+        scale="0.001 0.001 0.001" />
+            </xacro:if>
+            <xacro:if value="${'eli' in tip_sensor}">
               <!-- Ellispoid distal  -->
               <mesh filename="package://sr_description/hand/model/ellipsoids/distal_ellipsoid_visual.dae"
-		    scale="0.001 0.001 0.001" />
+        scale="0.001 0.001 0.001" />
             </xacro:if>
-            <xacro:unless value="${eli}">
-              <xacro:if value="${bio}">
-                <!-- biotac distal  -->
-                <mesh filename="package://sr_description/hand/model/F1.dae"
-                      scale="0.001 0.001 0.001" />
-              </xacro:if>
-              <xacro:unless value="${bio}">
-		<xacro:if value="${bt_sp}">
-                  <!-- bt_sp distal  -->
-                  <mesh filename="package://sr_description/hand/model/biotacs/sp.dae" />
-		</xacro:if>
-		<xacro:unless value="${bt_sp}">
-                  <!-- Standard distal  -->
-                  <mesh filename="package://sr_description/hand/model/F1.dae"
-			scale="0.001 0.001 0.001" />
-		</xacro:unless>
-              </xacro:unless>
-            </xacro:unless>
-          </xacro:unless>
+            <xacro:if value="${'bt_sp' in tip_sensor}">
+              <!-- bt_sp distal  -->
+              <mesh filename="package://sr_description/hand/model/biotacs/sp.dae" />
+            </xacro:if>
+          </xacro:if>
         </geometry>
         <material name="Grey" />
@@ -65,38 +53,29 @@
         <origin xyz="0 0 0" rpy="0 0 0" />
         <geometry name="${prefix}${link_prefix}distal_collision_geom">
-          <xacro:if value="${ubi}">
-            <!-- Ubi distal -->
-            <mesh filename="package://sr_description/hand/model/ubi_tactiles/ubi_tip_collision.dae"
-            scale="0.001 0.001 0.001" />
-          </xacro:if>
-          <xacro:unless value="${ubi}">
-            <xacro:if value="${eli}">
+          <xacro:if value="${tip_sensor in ['ubi','bt_sp','eli']}">
+            <xacro:if value="${'ubi' in tip_sensor}">
+              <!-- Ubi distal -->
+              <mesh filename="package://sr_description/hand/model/ubi_tactiles/ubi_tip_collision.dae"
+                    scale="0.001 0.001 0.001" />
+            </xacro:if>
+            <xacro:if value="${'eli' in tip_sensor}">
               <!-- Ellispoid distal  -->
               <mesh filename="package://sr_description/hand/model/ellipsoids/distal_ellipsoid.dae"
-              scale="0.001 0.001 0.001" />
+                    scale="0.001 0.001 0.001" />
             </xacro:if>
-            <xacro:unless value="${eli}">
-              <xacro:if value="${bio}">
-                <!-- biotac distal  -->
-                <mesh filename="package://sr_description/hand/model/F1.dae"
-                scale="0.001 0.001 0.001" />
-              </xacro:if>
-              <xacro:unless value="${bio}">
-		<xacro:if value="${bt_sp}">
-                  <!-- bt_sp distal  -->
-                  <mesh filename="package://sr_description/hand/model/biotacs/sp.dae" />
-		</xacro:if>
-		<xacro:unless value="${bt_sp}">
-                  <!-- Standard distal  -->
-                  <mesh filename="package://sr_description/hand/model/F1.dae"
-			scale="0.001 0.001 0.001" />
-		</xacro:unless>
-              </xacro:unless>
-            </xacro:unless>
+            <xacro:if value="${'bt_sp' in tip_sensor}">
+              <!-- bt_sp distal  -->
+              <mesh filename="package://sr_description/hand/model/biotacs/sp.dae" />
+            </xacro:if>
+          </xacro:if>
+          <xacro:unless value="${tip_sensor in ['ubi','bt_sp','eli']}">
+            <!-- Standard distal  -->
+            <mesh filename="package://sr_description/hand/model/F1.dae"
+                  scale="0.001 0.001 0.001" />
           </xacro:unless>
         </geometry>
       </collision>
     </link>
-    <xacro:unless value="${bio}">
+    <xacro:unless value="${'bio' in tip_sensor}">
       <joint name="${prefix}${joint_prefix}J1" type="revolute">
         <parent link="${parent}" />
@@ -134,6 +113,5 @@
     </xacro:unless>
     <!-- extensions -->
-    <xacro:distal_gazebo prefix="${prefix}"
-    link_prefix="${link_prefix}" />
+    <xacro:distal_gazebo />
   </xacro:macro>
 </robot>

File: sr_description/hand/xacro/finger/fingers.urdf.xacro (robot description, xacro)
@@ -8,8 +8,7 @@
   <!-- muscletrans is true for muscle transmission to be used, false to use motor transmission -->
   <!-- lf is true for little finger or false for standard finger -->
-  <!-- bio is true for biotac finger or false for standard finger -->
-  <!-- bt_sp is true for BT_SP finger or false for standard finger -->
-  <!-- ubi is true for ubi finger or false for standard finger -->
-  <!-- eli is true for ellipsoid fingertip or false for standard finger -->
+  <!-- tip_sensor describes the sensor none, bio, bt_sp, ubi, eli -->
+  <!-- mid_sensor describes the sensor none, bio, ubi -->
+  <!-- prox_sensor describes the sensor none, standard, ubi -->
   <!-- reflect is either 1 (for right hand) or -1 (for left hand) -->
   <!-- prefix can be anything but usually is "r_" or  "l_" for right and left hands distinction -->
@@ -18,50 +17,35 @@
   <!-- parent is the parent link for the first joint -->
   <xacro:macro name="finger"
-  params="muscletrans lf bio bt_sp ubi eli reflect prefix link_prefix joint_prefix parent *origin *axis">
+  params="muscletrans:=^ tip_sensor:=^|standard mid_sensor:=^|standard prox_sensor:=^|standard reflect:=^ prefix:=^ link_prefix joint_prefix parent *origin *axis">
     <!-- Little finger special case -->
-    <xacro:if value="${lf}">
-      <xacro:lfmetacarpal muscle="${muscletrans}"
-      prefix="${prefix}" reflect="${reflect}" parent="${parent}" />
+    <xacro:if value="${'lf' in link_prefix}">
+      <xacro:lfmetacarpal muscle="${muscletrans}" parent="${parent}" />
       <!-- Knuckle -->
-      <xacro:knuckle muscle="${muscletrans}" prefix="${prefix}"
-      link_prefix="${link_prefix}" joint_prefix="${joint_prefix}"
-      parent="${prefix}lfmetacarpal">
+      <xacro:knuckle muscle="${muscletrans}" parent="${prefix}lfmetacarpal">
         <xacro:insert_block name="origin" />
       </xacro:knuckle>
     </xacro:if>
     <!-- Standard finger -->
-    <xacro:unless value="${lf}">
+    <xacro:unless value="${'lf' in link_prefix}">
       <!-- Knuckle -->
-      <xacro:knuckle muscle="${muscletrans}" prefix="${prefix}"
-      link_prefix="${link_prefix}" joint_prefix="${joint_prefix}"
-      parent="${parent}">
+      <xacro:knuckle muscle="${muscletrans}" parent="${parent}">
         <xacro:insert_block name="origin" />
       </xacro:knuckle>
     </xacro:unless>
     <!-- Proximal -->
-    <xacro:proximal muscle="${muscletrans}" prefix="${prefix}"
-    link_prefix="${link_prefix}" joint_prefix="${joint_prefix}"
-    parent="${prefix}${link_prefix}knuckle"></xacro:proximal>
+    <xacro:proximal muscle="${muscletrans}" parent="${prefix}${link_prefix}knuckle"></xacro:proximal>
     <!-- Biotac Middle -->
-    <xacro:if value="${bio}">
-      <xacro:biotac_middle muscle="${muscletrans}"
-      prefix="${prefix}" link_prefix="${link_prefix}"
-      joint_prefix="${joint_prefix}"
-      parent="${prefix}${link_prefix}proximal">
+    <xacro:if value="${'bio' in tip_sensor}">
+      <xacro:biotac_middle muscle="${muscletrans}" parent="${prefix}${link_prefix}proximal">
       </xacro:biotac_middle>
     </xacro:if>
     <!-- Standard Middle -->
-    <xacro:unless value="${bio}">
-      <xacro:middle muscle="${muscletrans}" prefix="${prefix}"
-      link_prefix="${link_prefix}" joint_prefix="${joint_prefix}"
-      parent="${prefix}${link_prefix}proximal"></xacro:middle>
+    <xacro:unless value="${'bio' in tip_sensor}">
+      <xacro:middle muscle="${muscletrans}" parent="${prefix}${link_prefix}proximal"></xacro:middle>
     </xacro:unless>
     <!-- Distal  -->
     <!-- only if finger is not biotac  -->
-    <xacro:unless value="${bio}">
-      <xacro:distal muscle="${muscletrans}" bio="${bio}" bt_sp="${bt_sp}"
-      ubi="${ubi}" eli="${eli}" prefix="${prefix}"
-      link_prefix="${link_prefix}" joint_prefix="${joint_prefix}"
-      parent="${prefix}${link_prefix}middle"></xacro:distal>
+    <xacro:unless value="${'bio' in tip_sensor}">
+      <xacro:distal muscle="${muscletrans}" parent="${prefix}${link_prefix}middle"></xacro:distal>
     </xacro:unless>
   </xacro:macro>

File: sr_description/hand/xacro/finger/knuckle/knuckle.transmission.xacro (robot description, xacro)
@@ -8,5 +8,5 @@
     <!-- link_prefix prepends fingername to the link names -->
     <!-- joint_prefix prepends fingername to the joint names -->
-    <xacro:macro name="knuckle_transmission" params="muscletrans prefix joint_prefix link_prefix">
+    <xacro:macro name="knuckle_transmission" params="muscletrans:=^ prefix:=^ joint_prefix:=^ link_prefix:=^">
         <!-- muscle hand -->
         <xacro:if value="${muscletrans}">

File: sr_description/hand/xacro/finger/knuckle/knuckle.urdf.xacro (robot description, xacro)
@@ -14,5 +14,5 @@
   <!-- parent is the parent link for the joint -->
   <xacro:macro name="knuckle"
-  params="muscle prefix link_prefix joint_prefix parent *origin">
+  params="muscle:=^ prefix:=^ link_prefix:=^ joint_prefix:=^ parent *origin">
     <link name="${prefix}${link_prefix}knuckle">
       <inertial>
@@ -52,9 +52,6 @@
     </gazebo>
     <!-- extensions -->
-    <xacro:knuckle_transmission muscletrans="${muscle}"
-    prefix="${prefix}" joint_prefix="${joint_prefix}"
-    link_prefix="${link_prefix}" />
-    <xacro:knuckle_gazebo prefix="${prefix}"
-    link_prefix="${link_prefix}" />
+    <xacro:knuckle_transmission muscletrans="${muscle}" />
+    <xacro:knuckle_gazebo />
   </xacro:macro>
 </robot>
