Commit message: Support sensor selection, to permit deactivating gazebo sensors and simplified xacro docs using latest xacro features

File: sr_description/hand/xacro/finger/lfmetacarpal/lfmetacarpal.gazebo.xacro (robot description, xacro)
@@ -1,21 +1,23 @@
 <?xml version="1.0"?>
 <robot xmlns:xacro="http://www.ros.org/wiki/xacro">
-  <xacro:macro name="lfmetacarpal_gazebo" params="prefix link_prefix">
-  <!-- prefix can be anything but usually is "r_" or  "l_" for right and left hands distinction -->
-  <gazebo reference="${prefix}lfmetacarpal">
-      <sensor type="contact" name="${prefix}lfmetacarpal_contact">
-				<always_on>1</always_on>
-        <update_rate>1000.0</update_rate>
-        <contact>
-          <collision>${prefix}lfmetacarpal_collision</collision>
-          <topic>${prefix}lfmetacarpal_collision</topic>
-        </contact>
-        <plugin name="${prefix}lfmetacarpal_gazebo_ros_bumper_controller" filename="libgazebo_ros_bumper.so">
-          <alwaysOn>true</alwaysOn>
-          <frameName>${prefix}lfmetacarpal</frameName>
-          <updateRate>100.0</updateRate>
-          <bumperTopicName>contacts/${prefix}lf/metacarpal</bumperTopicName>
-        </plugin>
-      </sensor>
+  <xacro:macro name="lfmetacarpal_gazebo" params="prefix:=^ palm_sensor:=^|bumper link_prefix">
+    <!-- prefix can be anything but usually is "r_" or  "l_" for right and left hands distinction -->
+    <gazebo reference="${prefix}lfmetacarpal">
+      <xacro:unless value="${'none' in palm_sensor}" >
+        <sensor type="contact" name="${prefix}lfmetacarpal_contact">
+          <always_on>1</always_on>
+          <update_rate>1000.0</update_rate>
+          <contact>
+            <collision>${prefix}lfmetacarpal_collision</collision>
+            <topic>${prefix}lfmetacarpal_collision</topic>
+          </contact>
+          <plugin name="${prefix}lfmetacarpal_gazebo_ros_bumper_controller" filename="libgazebo_ros_bumper.so">
+            <alwaysOn>true</alwaysOn>
+            <frameName>${prefix}lfmetacarpal</frameName>
+            <updateRate>100.0</updateRate>
+            <bumperTopicName>contacts/${prefix}lf/metacarpal</bumperTopicName>
+          </plugin>
+        </sensor>
+        </xacro:unless>
       <selfCollide>true</selfCollide>
     </gazebo>

File: sr_description/hand/xacro/finger/lfmetacarpal/lfmetacarpal.transmission.xacro (robot description, xacro)
@@ -6,5 +6,5 @@
     <!-- muscletrans is true for muscle transmission or false for motor transmission -->
     <!-- prefix can be anything but usually is "r_" or  "l_" for right and left hands distinction -->
-    <xacro:macro name="lfmetacarpal_transmission" params="muscletrans prefix">
+    <xacro:macro name="lfmetacarpal_transmission" params="muscletrans prefix:=^">
         <!-- muscle hand -->
         <xacro:if value="${muscletrans}">

File: sr_description/hand/xacro/finger/lfmetacarpal/lfmetacarpal.urdf.xacro (robot description, xacro)
@@ -13,5 +13,5 @@
   <!-- parent is the parent link for the joint -->
   <xacro:macro name="lfmetacarpal"
-  params="muscle prefix reflect parent">
+  params="muscle:=^ prefix:=^ reflect:=^ parent">
     <link name="${prefix}lfmetacarpal">
       <inertial>
@@ -50,8 +50,6 @@
     </gazebo>
     <!-- extensions -->
-    <xacro:lfmetacarpal_transmission muscletrans="${muscle}"
-    prefix="${prefix}" />
-    <xacro:lfmetacarpal_gazebo prefix="${prefix}"
-    link_prefix="${link_prefix}" />
+    <xacro:lfmetacarpal_transmission muscletrans="${muscle}"/>
+    <xacro:lfmetacarpal_gazebo link_prefix="${link_prefix}" />
   </xacro:macro>
 </robot>

File: sr_description/hand/xacro/finger/middle/middle.gazebo.xacro (robot description, xacro)
@@ -1,7 +1,8 @@
 <?xml version="1.0"?>
 <robot xmlns:xacro="http://www.ros.org/wiki/xacro">
-  <xacro:macro name="middle_gazebo" params="prefix link_prefix">
-  <!-- prefix can be anything but usually is "r_" or  "l_" for right and left hands distinction -->
-  <gazebo reference="${prefix}${link_prefix}middle">
+  <xacro:macro name="middle_gazebo" params="prefix:=^ link_prefix:=^ mid_sensor:=^|bumper">
+    <!-- prefix can be anything but usually is "r_" or  "l_" for right and left hands distinction -->
+    <gazebo reference="${prefix}${link_prefix}middle">
+      <xacro:unless value="${'none' in mid_sensor}">
       <sensor type="contact" name="${prefix}${link_prefix}middle_contact">
         <always_on>1</always_on>
@@ -18,4 +19,5 @@
         </plugin>
       </sensor>
+      </xacro:unless>
       <selfCollide>true</selfCollide>
     </gazebo>

File: sr_description/hand/xacro/finger/middle/middle.transmission.xacro (robot description, xacro)
@@ -8,5 +8,5 @@
     <!-- link_prefix prepends fingername to the link names -->
     <!-- joint_prefix prepends fingername to the joint names -->
-    <xacro:macro name="middle_transmission" params="muscletrans prefix joint_prefix link_prefix">
+    <xacro:macro name="middle_transmission" params="muscletrans:=^ prefix:=^ joint_prefix:=^ link_prefix:=^">
         <!-- muscle hand -->
         <xacro:if value="${muscletrans}">

File: sr_description/hand/xacro/finger/middle/middle.urdf.xacro (robot description, xacro)
@@ -14,5 +14,5 @@
   <!-- parent is the parent link for the joint -->
   <xacro:macro name="middle"
-  params="muscle prefix link_prefix joint_prefix parent">
+  params="muscle:=^ prefix:=^ link_prefix:=^ joint_prefix:=^ parent">
     <link name="${prefix}${link_prefix}middle">
       <inertial>
@@ -63,9 +63,6 @@
     </gazebo>
     <!-- extensions -->
-    <xacro:middle_transmission muscletrans="${muscle}"
-    prefix="${prefix}" joint_prefix="${joint_prefix}"
-    link_prefix="${link_prefix}" />
-    <xacro:middle_gazebo prefix="${prefix}"
-    link_prefix="${link_prefix}" />
+    <xacro:middle_transmission muscletrans="${muscle}" />
+    <xacro:middle_gazebo />
   </xacro:macro>
 </robot>

File: sr_description/hand/xacro/finger/proximal/proximal.gazebo.xacro (robot description, xacro)
@@ -1,7 +1,8 @@
 <?xml version="1.0"?>
 <robot xmlns:xacro="http://www.ros.org/wiki/xacro">
-  <xacro:macro name="proximal_gazebo" params="prefix link_prefix">
-  <!-- prefix can be anything but usually is "r_" or  "l_" for right and left hands distinction -->
-  <gazebo reference="${prefix}${link_prefix}proximal">
+  <xacro:macro name="proximal_gazebo" params="prefix:=^ link_prefix:=^ prox_sensor:=^|standard">
+    <!-- prefix can be anything but usually is "r_" or  "l_" for right and left hands distinction -->
+    <gazebo reference="${prefix}${link_prefix}proximal">
+      <xacro:unless value="${'none' in prox_sensor}" >
       <sensor type="contact" name="${prefix}${link_prefix}proximal_contact">
         <always_on>1</always_on>
@@ -18,4 +19,5 @@
         </plugin>
       </sensor>
+      </xacro:unless>
       <selfCollide>true</selfCollide>
     </gazebo>

File: sr_description/hand/xacro/finger/proximal/proximal.transmission.xacro (robot description, xacro)
@@ -8,5 +8,5 @@
     <!-- link_prefix prepends fingername to the link names -->
     <!-- joint_prefix prepends fingername to the joint names -->
-    <xacro:macro name="proximal_transmission" params="muscletrans prefix joint_prefix link_prefix">
+    <xacro:macro name="proximal_transmission" params="muscletrans:=^ prefix:=^ joint_prefix:=^ link_prefix:=^">
         <!-- muscle hand -->
         <xacro:if value="${muscletrans}">

File: sr_description/hand/xacro/finger/proximal/proximal.urdf.xacro (robot description, xacro)
@@ -14,5 +14,5 @@
   <!-- parent is the parent link for the joint -->
   <xacro:macro name="proximal"
-  params="muscle prefix link_prefix joint_prefix parent">
+  params="muscle:=^ prefix:=^ link_prefix:=^ joint_prefix:=^ parent">
     <link name="${prefix}${link_prefix}proximal">
       <inertial>
@@ -51,9 +51,6 @@
     </gazebo>
     <!-- extensions -->
-    <xacro:proximal_transmission muscletrans="${muscle}"
-    prefix="${prefix}" joint_prefix="${joint_prefix}"
-    link_prefix="${link_prefix}" />
-    <xacro:proximal_gazebo prefix="${prefix}"
-    link_prefix="${link_prefix}" />
+    <xacro:proximal_transmission muscletrans="${muscle}" />
+    <xacro:proximal_gazebo />
   </xacro:macro>
 </robot>

File: sr_description/hand/xacro/forearm/forearm.urdf.xacro (robot description, xacro)
@@ -2,5 +2,5 @@
   <!-- muscle is true for muscle hand or false for motor hand -->
   <!-- prefix can be anything but usually is "r_" or  "l_" for right and left hands distinction -->
-  <xacro:macro name="forearm" params="muscle prefix">
+  <xacro:macro name="forearm" params="muscle:=^ prefix:=^">
     <link name="${prefix}forearm">
       <inertial>

File: sr_description/hand/xacro/forearm/forearm_lite.urdf.xacro (robot description, xacro)
@@ -2,5 +2,5 @@
   <!-- muscle is true for muscle hand or false for motor hand -->
   <!-- prefix can be anything but usually is "r_" or  "l_" for right and left hands distinction -->
-  <xacro:macro name="forearm" params="muscle prefix">
+  <xacro:macro name="forearm" params="muscle:=^ prefix:=^">
     <link name="${prefix}forearm">
       <inertial>

File: sr_description/hand/xacro/full_hand.urdf.xacro (robot description, xacro)
@@ -11,52 +11,45 @@
   <!-- muscletrans is true for muscle transmission to be used, false to use motor transmission -->
   <!-- muscle is true for muscle hand or false for motor hand -->
-  <!-- bio is true for biotac finger or false for standard finger -->
-  <!-- bt_sp is true for BT_SP finger or false for standard finger -->
-  <!-- ubi is true for ubi finger or false for standard finger -->
-  <!-- eli is true for ellipsoid fingertip or false for standard finger -->
+  <!-- bio (deprecated) is true for biotac finger or false for standard finger -->
+  <!-- bt_sp (deprecated) is true for BT_SP finger or false for standard finger -->
+  <!-- ubi (deprecated) is true for ubi finger or false for standard finger -->
+  <!-- eli (deprecated) is true for ellipsoid fingertip or false for standard finger -->
+  <!-- tip_sensor describes the sensor none, bio, bt_sp, ubi, eli -->
+  <!-- mid_sensor describes the sensor none, bio, ubi -->
+  <!-- prox_sensor describes the sensor none, bumper, ubi -->
+  <!-- palm_sensor describes the sensor none, bumper, ubi -->
   <!-- reflect is either 1 (for right hand) or -1 (for left hand) -->
   <!-- prefix can be anything but usually is "r_" or  "l_" for right and left hands distinction -->
   <!-- lf is true if we want a little finger, false otherwise -->
   <xacro:macro name="shadowhand"
-  params="muscletrans muscle bio bt_sp ubi eli reflect prefix lf">
+  params="muscletrans muscle bio:=False bt_sp:=False ubi:=False eli:=False tip_sensor:=standard prox_sensor:=standard mid_sensor:=standard palm_sensor:=standard reflect prefix lf">
+    <xacro:include filename="$(find sr_description)/hand/xacro/backward_compat.urdf.xacro" />
     <!-- Forearm -->
-    <xacro:forearm muscle="${muscle}" prefix="${prefix}" />
+    <xacro:forearm />
     <!-- Wrist -->
     <xacro:if value="${muscle}">
-      <xacro:wrist muscletrans="${muscletrans}" prefix="${prefix}"
-      reflect="${reflect}" parent="${prefix}forearm">
+      <xacro:wrist parent="${prefix}forearm">
         <origin xyz="0 0 0.4096" rpy="0 0 0" />
       </xacro:wrist>
     </xacro:if>
     <xacro:unless value="${muscle}">
-      <xacro:wrist muscletrans="false" prefix="${prefix}"
-      reflect="${reflect}" parent="${prefix}forearm">
+      <xacro:wrist muscletrans="false" parent="${prefix}forearm">
         <origin xyz="0 -0.010 0.213" rpy="0 0 0" />
       </xacro:wrist>
     </xacro:unless>
     <!-- Palm -->
-    <xacro:palm muscletrans="${muscletrans}" prefix="${prefix}"
-    reflect="${reflect}" parent="${prefix}wrist" />
+    <xacro:palm parent="${prefix}wrist" />
     <!-- First Finger -->
-    <xacro:finger muscletrans="${muscletrans}" lf="false"
-    bio="${bio}" bt_sp="${bt_sp}" ubi="${ubi}" eli="${eli}" prefix="${prefix}"
-    reflect="${reflect}" link_prefix="ff" joint_prefix="FF"
-    parent="${prefix}palm">
+    <xacro:finger link_prefix="ff" joint_prefix="FF" parent="${prefix}palm">
       <origin xyz="${reflect*0.033} 0 0.095" rpy="0 0 0" />
       <axis xyz="0 ${-1*reflect} 0" />
     </xacro:finger>
     <!-- Middle Finger -->
-    <xacro:finger muscletrans="${muscletrans}" lf="false"
-    bio="${bio}" bt_sp="${bt_sp}" ubi="${ubi}" eli="${eli}" prefix="${prefix}"
-    reflect="${reflect}" link_prefix="mf" joint_prefix="MF"
-    parent="${prefix}palm">
+    <xacro:finger link_prefix="mf" joint_prefix="MF" parent="${prefix}palm">
       <origin xyz="${reflect*0.011} 0 0.099" rpy="0 0 0" />
       <axis xyz="0 ${-1*reflect} 0" />
     </xacro:finger>
     <!-- Ring Finger -->
-    <xacro:finger muscletrans="${muscletrans}" lf="false"
-    bio="${bio}" bt_sp="${bt_sp}" ubi="${ubi}" eli="${eli}" prefix="${prefix}"
-    reflect="${reflect}" link_prefix="rf" joint_prefix="RF"
-    parent="${prefix}palm">
+    <xacro:finger link_prefix="rf" joint_prefix="RF" parent="${prefix}palm">
       <origin xyz="${reflect*-0.011} 0 0.095" rpy="0 0 0" />
       <axis xyz="0 ${reflect} 0" />
@@ -64,8 +57,5 @@
     <!-- Little Finger  -->
     <xacro:if value="${lf}">
-      <xacro:finger muscletrans="${muscletrans}" lf="true"
-      bio="${bio}" bt_sp="${bt_sp}" ubi="${ubi}" eli="${eli}" prefix="${prefix}"
-      reflect="${reflect}" link_prefix="lf" joint_prefix="LF"
-      parent="${prefix}palm">
+      <xacro:finger link_prefix="lf" joint_prefix="LF" parent="${prefix}palm">
         <origin xyz="0 0 0.06579" rpy="0 0 0" />
         <axis xyz="0 ${reflect} 0" />
@@ -73,8 +63,5 @@
     </xacro:if>
     <!-- Thumb  -->
-    <xacro:thumb muscletrans="${muscletrans}" bio="${bio}" bt_sp="${bt_sp}"
-    ubi="${ubi}" eli="${eli}" prefix="${prefix}"
-    reflect="${reflect}" is_lite="0" parent="${prefix}palm">
-    </xacro:thumb>
+    <xacro:thumb is_lite="0" parent="${prefix}palm" />
   </xacro:macro>
 </robot>
