Commit message: add a child element called imu, to be compatible with SensorParser, and avoid xacro breaking by renaming macro to imu_sensor

File: sr_description/hand/xacro/palm/imu.urdf.xacro (robot description, xacro)
@@ -1,4 +1,4 @@
 <robot xmlns:xacro="http://www.ros.org/wiki/xacro" name="shadowhand_motor">
-  <xacro:macro name="imu" params="prefix">
+  <xacro:macro name="imu_sensor" params="prefix">
     <link name="${prefix}imu"/>
     <joint name="${prefix}palm_to_imu" type="fixed">
@@ -7,7 +7,8 @@
       <origin xyz="0.01785 0.00765 0.049125" rpy="-1.5707963 3.141592 0.0"/>
     </joint>
-    <sensor name="${prefix}imu" update_rate="100">
+    <sensor name="${prefix}imu" update_rate="100" >
       <parent link="${prefix}imu"/>
       <origin xyz="0 0 0" rpy="0 0 0"/>
+      <imu />
     </sensor>
   </xacro:macro>

File: sr_description/hand/xacro/palm/palm.urdf.xacro (robot description, xacro)
@@ -108,5 +108,5 @@
     </gazebo>
     <!--imu-->
-    <xacro:imu prefix="${prefix}"/>
+    <xacro:imu_sensor prefix="${prefix}"/>
     <!-- extensions -->
     <xacro:shadowhand_palm_transmission muscletrans="${muscletrans}"

File: sr_description/hand/xacro/palm/palm_lite.urdf.xacro (robot description, xacro)
@@ -88,5 +88,5 @@
     <!-- No wrist joints in a Lite palm -->
     <!-- extensions -->
-    <xacro:imu prefix="${prefix}" />
+    <xacro:imu_sensor prefix="${prefix}" />
     <xacro:shadowhand_palm_gazebo prefix="${prefix}" />
   </xacro:macro>
